File: hardware/sheets/matrix_rows.kicad_sch (KiCad schematic)
At the start: 0 parts

Commit message: hw: draw matrix driver and LED matrix sheets
Columns: two cascaded TLC59283 sinks on 3V3. R_IREF is 2.94k, an
18.0 mA nominal setting (about 19.4 mA worst case with driver and
resistor tolerance), with a fitted 0 ohm in series, so adjustment can
only lower the current.

Rows: the TLC chain output, clock, latch and SAFE cross into the LED
rail through an SN74LVC8T245 translator. Four SN74HC595 on VLED drive
32 AO3401A high-side switches with 10k gate pull-ups, with row
pull-downs as unfitted options.

Scan-stall safety: every latch retriggers an SN74LVC1G123. TI
specifies 1.0-1.1 ms at 10k / 0.1 uF; with the fitted parts'
tolerances the timeout is 0.76-1.41 ms. The part has only a Q
output, so an inverter makes SAFE = NOT Q. SAFE forces the column
BLANK through an OR gate and tri-states the row registers, and the
MCU reads it. The matrix stays dark while the MCU is off or in
reset.

LED matrix: 1024 LEDs, anodes on the rows and cathodes on the
columns, drawn as row and column buses, on the front side with the
buttons (ADR 0008).

The pending ERC exclusions for the matrix labels are removed. Four
reviewed exclusions cover the translator's unused inputs, which are
tied to ground as TI requires.
Parts:
- added C701, C702, C703, C704, C705, C706, C709, C710, C711, C712: 100nF, Capacitor_SMD:C_0402_1005Metric, symbol Device:C
- added C707, C708: 10uF 25V, Capacitor_SMD:C_0805_2012Metric, symbol Device:C
- added Q701, Q702, Q703, Q704, Q705, Q706, Q707, Q708, Q709, Q710, Q711, Q712, Q713, Q714, Q715, Q716, Q717, Q718, Q719, Q720, Q721, Q722, Q723, Q724, Q725, Q726, Q727, Q728, Q729, Q730, Q731, Q732: AO3401A, Package_TO_SOT_SMD:SOT-23, symbol Transistor_FET:AO3401A
- added R701: 0, Resistor_SMD:R_0402_1005Metric, symbol Device:R
- added R702: 10k, Resistor_SMD:R_0402_1005Metric, symbol Device:R
- added R703, R704: 100k, Resistor_SMD:R_0402_1005Metric, symbol Device:R
- added RN701, RN702, RN703, RN704, RN705, RN706, RN707, RN708: 4x10k, Resistor_SMD:R_Array_Convex_4x0603, symbol Device:R_Pack04
- added RN709, RN710, RN711, RN712, RN713, RN714, RN715, RN716: DNP, Resistor_SMD:R_Array_Convex_4x0603, symbol Device:R_Pack04
- added TP701: MTX_BLANK, TestPoint:TestPoint_Pad_D1.0mm, symbol Connector:TestPoint
- added TP702: BLANK_TLC, TestPoint:TestPoint_Pad_D1.0mm, symbol Connector:TestPoint
- added TP703: MTX_SAFE_SENSE, TestPoint:TestPoint_Pad_D1.0mm, symbol Connector:TestPoint
- added TP704: SCAN_OK, TestPoint:TestPoint_Pad_D1.0mm, symbol Connector:TestPoint
- added TP705: SER_V, TestPoint:TestPoint_Pad_D1.0mm, symbol Connector:TestPoint
- added TP706: SRCLK_V, TestPoint:TestPoint_Pad_D1.0mm, symbol Connector:TestPoint
- added TP707: RCLK_V, TestPoint:TestPoint_Pad_D1.0mm, symbol Connector:TestPoint
- added TP708: ROW0, TestPoint:TestPoint_Pad_D1.0mm, symbol Connector:TestPoint
- added TP709: ROW16, TestPoint:TestPoint_Pad_D1.0mm, symbol Connector:TestPoint
- added TP710: ROW31, TestPoint:TestPoint_Pad_D1.0mm, symbol Connector:TestPoint
- added U701: SN74LVC8T245, Package_SO:TSSOP-24_4.4x7.8mm_P0.65mm, symbol Logic_LevelTranslator:SN74LVC8T245
- added U702, U703, U704, U705: SN74HC595, Package_SO:TSSOP-16_4.4x5mm_P0.65mm, symbol 74xx:74HC595
- added U706: SN74LVC1G123, Package_SO:SSOP-8_2.95x2.8mm_P0.65mm, symbol smart-led-badge:SN74LVC1G123
- added U707: SN74LVC1G04, Package_TO_SOT_SMD:SOT-23-5, symbol 74xGxx:74LVC1G04
- added U708: SN74LVC1G32, Package_TO_SOT_SMD:SOT-23-5, symbol 74xGxx:74LVC1G32
Connections:
- new net +3V3: C701.1, C710.1, C711.1, C712.1, R702.2, R704.2, U701.1 (V_{CCA}), U701.2 (DIR), U706.8 (VCC), U707.5 (VCC), U708.5 (VCC)
- new net BLANK_TLC: TP702.1, U708.4
- new net GND: C701.2, C702.2, C703.2, C704.2, C705.2, C706.2, C707.2, C708.2, C710.2, C711.2, C712.2, R701.2, R703.2, RN709.5 (R4.2), RN709.6 (R3.2), RN709.7 (R2.2), RN709.8 (R1.2), RN710.5 (R4.2), RN710.6 (R3.2), RN710.7 (R2.2), RN710.8 (R1.2), RN711.5 (R4.2), RN711.6 (R3.2), RN711.7 (R2.2), RN711.8 (R1.2), RN712.5 (R4.2), RN712.6 (R3.2), RN712.7 (R2.2), RN712.8 (R1.2), RN713.5 (R4.2), RN713.6 (R3.2), RN713.7 (R2.2), RN713.8 (R1.2), RN714.5 (R4.2), RN714.6 (R3.2), RN714.7 (R2.2), RN714.8 (R1.2), RN715.5 (R4.2), RN715.6 (R3.2), RN715.7 (R2.2), RN715.8 (R1.2), RN716.5 (R4.2), RN716.6 (R3.2), RN716.7 (R2.2), RN716.8 (R1.2), U701.10 (A8), U701.11 (GND), U701.12 (GND), U701.13 (GND), U701.7 (A5), U701.8 (A6), U701.9 (A7), U702.8 (GND), U703.8 (GND), U704.8 (GND), U705.8 (GND), U706.1 (~{A}), U706.4 (GND), U707.3 (GND), U708.3 (GND)
- new net MONO_CEXT: C709.1, U706.6 (Cext)
- new net MONO_RCEXT: C709.2, R702.1, U706.7 (Rext/Cext)
- new net MTX_ARM: R703.1, U706.3 (~{CLR})
- new net MTX_BLANK: R704.1, TP701.1, U708.1
- new net MTX_LAT: U701.5 (A3), U706.2 (B)
- new net MTX_MISO: U701.3 (A1)
- new net MTX_SAFE_SENSE: TP703.1, U701.6 (A4), U707.4, U708.2
- new net MTX_SCK: U701.4 (A2)
- new net OE_V: U701.18 (B4), U702.13 (~{OE}), U703.13 (~{OE}), U704.13 (~{OE}), U705.13 (~{OE})
- new net RCLK_V: TP707.1, U701.19 (B3), U702.12 (RCLK), U703.12 (RCLK), U704.12 (RCLK), U705.12 (RCLK)
- new net RG0: Q701.1 (G), RN701.1 (R1.1), U702.15 (QA)
- new net RG1: Q702.1 (G), RN701.2 (R2.1), U702.1 (QB)
- new net RG10: Q711.1 (G), RN703.3 (R3.1), U703.2 (QC)
- new net RG11: Q712.1 (G), RN703.4 (R4.1), U703.3 (QD)
- new net RG12: Q713.1 (G), RN704.1 (R1.1), U703.4 (QE)
- new net RG13: Q714.1 (G), RN704.2 (R2.1), U703.5 (QF)
- new net RG14: Q715.1 (G), RN704.3 (R3.1), U703.6 (QG)
- new net RG15: Q716.1 (G), RN704.4 (R4.1), U703.7 (QH)
- new net RG16: Q717.1 (G), RN705.1 (R1.1), U704.15 (QA)
- new net RG17: Q718.1 (G), RN705.2 (R2.1), U704.1 (QB)
- new net RG18: Q719.1 (G), RN705.3 (R3.1), U704.2 (QC)
- new net RG19: Q720.1 (G), RN705.4 (R4.1), U704.3 (QD)
- new net RG2: Q703.1 (G), RN701.3 (R3.1), U702.2 (QC)
- new net RG20: Q721.1 (G), RN706.1 (R1.1), U704.4 (QE)
- new net RG21: Q722.1 (G), RN706.2 (R2.1), U704.5 (QF)
- new net RG22: Q723.1 (G), RN706.3 (R3.1), U704.6 (QG)
- new net RG23: Q724.1 (G), RN706.4 (R4.1), U704.7 (QH)
- new net RG24: Q725.1 (G), RN707.1 (R1.1), U705.15 (QA)
- new net RG25: Q726.1 (G), RN707.2 (R2.1), U705.1 (QB)
- new net RG26: Q727.1 (G), RN707.3 (R3.1), U705.2 (QC)
- new net RG27: Q728.1 (G), RN707.4 (R4.1), U705.3 (QD)
- new net RG28: Q729.1 (G), RN708.1 (R1.1), U705.4 (QE)
- new net RG29: Q730.1 (G), RN708.2 (R2.1), U705.5 (QF)
- new net RG3: Q704.1 (G), RN701.4 (R4.1), U702.3 (QD)
- new net RG30: Q731.1 (G), RN708.3 (R3.1), U705.6 (QG)
- new net RG31: Q732.1 (G), RN708.4 (R4.1), U705.7 (QH)
- new net RG4: Q705.1 (G), RN702.1 (R1.1), U702.4 (QE)
- new net RG5: Q706.1 (G), RN702.2 (R2.1), U702.5 (QF)
- new net RG6: Q707.1 (G), RN702.3 (R3.1), U702.6 (QG)
- new net RG7: Q708.1 (G), RN702.4 (R4.1), U702.7 (QH)
- new net RG8: Q709.1 (G), RN703.1 (R1.1), U703.15 (QA)
- new net RG9: Q710.1 (G), RN703.2 (R2.1), U703.1 (QB)
- new net ROW0: Q701.3 (D), RN709.1 (R1.1), TP708.1
- new net ROW1: Q702.3 (D), RN709.2 (R2.1)
- new net ROW10: Q711.3 (D), RN711.3 (R3.1)
- new net ROW11: Q712.3 (D), RN711.4 (R4.1)
- new net ROW12: Q713.3 (D), RN712.1 (R1.1)
- new net ROW13: Q714.3 (D), RN712.2 (R2.1)
- new net ROW14: Q715.3 (D), RN712.3 (R3.1)
- new net ROW15: Q716.3 (D), RN712.4 (R4.1)
- new net ROW16: Q717.3 (D), RN713.1 (R1.1), TP709.1
- new net ROW17: Q718.3 (D), RN713.2 (R2.1)
- new net ROW18: Q719.3 (D), RN713.3 (R3.1)
- new net ROW19: Q720.3 (D), RN713.4 (R4.1)
- new net ROW2: Q703.3 (D), RN709.3 (R3.1)
- new net ROW20: Q721.3 (D), RN714.1 (R1.1)
- new net ROW21: Q722.3 (D), RN714.2 (R2.1)
- new net ROW22: Q723.3 (D), RN714.3 (R3.1)
- new net ROW23: Q724.3 (D), RN714.4 (R4.1)
- new net ROW24: Q725.3 (D), RN715.1 (R1.1)
- new net ROW25: Q726.3 (D), RN715.2 (R2.1)
- new net ROW26: Q727.3 (D), RN715.3 (R3.1)
- new net ROW27: Q728.3 (D), RN715.4 (R4.1)
- new net ROW28: Q729.3 (D), RN716.1 (R1.1)
- new net ROW29: Q730.3 (D), RN716.2 (R2.1)
- new net ROW3: Q704.3 (D), RN709.4 (R4.1)
- new net ROW30: Q731.3 (D), RN716.3 (R3.1)
- new net ROW31: Q732.3 (D), RN716.4 (R4.1), TP710.1
- new net ROW4: Q705.3 (D), RN710.1 (R1.1)
- new net ROW5: Q706.3 (D), RN710.2 (R2.1)
- new net ROW6: Q707.3 (D), RN710.3 (R3.1)
- new net ROW7: Q708.3 (D), RN710.4 (R4.1)
- new net ROW8: Q709.3 (D), RN711.1 (R1.1)
- new net ROW9: Q710.3 (D), RN711.2 (R2.1)
- new net SCAN_OK: TP704.1, U706.5 (Q), U707.2
- new net SER1: U702.9 (QH'), U703.14 (SER)
- new net SER2: U703.9 (QH'), U704.14 (SER)
- new net SER3: U704.9 (QH'), U705.14 (SER)
- new net SER_V: TP705.1, U701.21 (B1), U702.14 (SER)
- new net SRCLK_V: TP706.1, U701.20 (B2), U702.11 (SRCLK), U703.11 (SRCLK), U704.11 (SRCLK), U705.11 (SRCLK)
- new net VLED: C702.1, C703.1, C704.1, C705.1, C706.1, C707.1, C708.1, Q701.2 (S), Q702.2 (S), Q703.2 (S), Q704.2 (S), Q705.2 (S), Q706.2 (S), Q707.2 (S), Q708.2 (S), Q709.2 (S), Q710.2 (S), Q711.2 (S), Q712.2 (S), Q713.2 (S), Q714.2 (S), Q715.2 (S), Q716.2 (S), Q717.2 (S), Q718.2 (S), Q719.2 (S), Q720.2 (S), Q721.2 (S), Q722.2 (S), Q723.2 (S), Q724.2 (S), Q725.2 (S), Q726.2 (S), Q727.2 (S), Q728.2 (S), Q729.2 (S), Q730.2 (S), Q731.2 (S), Q732.2 (S), RN701.5 (R4.2), RN701.6 (R3.2), RN701.7 (R2.2), RN701.8 (R1.2), RN702.5 (R4.2), RN702.6 (R3.2), RN702.7 (R2.2), RN702.8 (R1.2), RN703.5 (R4.2), RN703.6 (R3.2), RN703.7 (R2.2), RN703.8 (R1.2), RN704.5 (R4.2), RN704.6 (R3.2), RN704.7 (R2.2), RN704.8 (R1.2), RN705.5 (R4.2), RN705.6 (R3.2), RN705.7 (R2.2), RN705.8 (R1.2), RN706.5 (R4.2), RN706.6 (R3.2), RN706.7 (R2.2), RN706.8 (R1.2), RN707.5 (R4.2), RN707.6 (R3.2), RN707.7 (R2.2), RN707.8 (R1.2), RN708.5 (R4.2), RN708.6 (R3.2), RN708.7 (R2.2), RN708.8 (R1.2), U701.23 (V_{CCB}), U701.24 (V_{CCB}), U702.10 (~{SRCLR}), U702.16 (VCC), U703.10 (~{SRCLR}), U703.16 (VCC), U704.10 (~{SRCLR}), U704.16 (VCC), U705.10 (~{SRCLR}), U705.16 (VCC)
- new net XLAT_OE_N: R701.1, U701.22 (~{OE})
- no-connect marks 0 -> 5
Other:
- note added: "Matrix row drivers and scan-stall safety (Rev A) - design notes Row chain: TLC chain SOUT (MTX_MISO), MTX_SCK, MTX_LAT and SAFE cross into the VLED domain through U701 (SN74LVC8T245, VCCA 3V3, VCCB VLED, DIR high = A to B). Its VCC isolation and Ioff keep 3V3 signals off the unpowered 595s when the LED rail is off. 4 x SN74HC595 on VLED (VCC 2-6 V) shift 32 row bits behind the 32 column bits; one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"

Commit message: hw: pull the row-register OE line up to VLED
If 3V3 collapses while the LED rail is still charged, the translator
enters VCC isolation and its outputs go high-impedance, leaving the
74HC595 OE inputs floating. An enabled register could then keep a
PFET gate low. A 100k pull-up from OE_V to VLED holds the registers'
outputs off in that state, so the gate pull-ups turn every row off.
The translator drives OE_V normally.

The sheet notes also state the one-shot timing as TI's guaranteed
limits and the R x C scaling used for the component tolerances.
Parts:
- added R705: 100k, Resistor_SMD:R_0402_1005Metric, symbol Device:R
Connections:
- net OE_V: now also R705.1
- net VLED: now also R705.2
Changed lines of the file:
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@@
 		(comment 2 "Draft: schematic capture in progress, not for fabrication")
 	)
-	(text "Matrix row drivers and scan-stall safety (Rev A) - design notes\n\nRow chain: TLC chain SOUT (MTX_MISO), MTX_SCK, MTX_LAT and SAFE cross into the VLED domain through U701\n(SN74LVC8T245, VCCA 3V3, VCCB VLED, DIR high = A to B). Its VCC isolation and Ioff keep 3V3 signals off the\nunpowered 595s when the LED rail is off. 4 x SN74HC595 on VLED (VCC 2-6 V) shift 32 row bits behind the 32 column\nbits; one LAT edge updates rows and columns together. QA..QH drive AO3401A gates (S = VLED, D = ROWn) with 10k\npull-ups to VLED, so rows are off whenever the 595 outputs are Hi-Z. Row pull-downs are DNP options.\n\nScan-stall safety (REQ-L5), CPU-independent: U706 SN74LVC1G123 is retriggered by every MTX_LAT rising edge\n(A low, CLR = MTX_ARM). Q stays high while latches keep arriving. tw: TI spec 1.0-1.1 ms at Rext 10k / Cext 0.1 uF; with R 1%, C709 X7R\n+/-10% initial and +/-15% over temperature 0.76-1.41 ms (DC bias only shortens it); measure on Rev A.\nThe 1G123 has only a Q output, so U707 inverts it: SAFE = NOT Q (net MTX_SAFE_SENSE, read by P0.21).\nSAFE high (stall, reset, MTX_ARM low) forces BLANK_TLC via U708 and tri-states the 595 outputs (OE_V), so all\nrows and columns turn off. MTX_BLANK pulled up and MTX_ARM pulled down keep the matrix dark with the MCU off.\nResidual: a firmware fault that keeps latching the same row is not caught here (column cap limits current).\nNothing measured."
+	(text "Matrix row drivers and scan-stall safety (Rev A) - design notes\n\nRow chain: TLC chain SOUT (MTX_MISO), MTX_SCK, MTX_LAT and SAFE cross into the VLED domain through U701\n(SN74LVC8T245, VCCA 3V3, VCCB VLED, DIR high = A to B). Its VCC isolation and Ioff keep 3V3 signals off the\nunpowered 595s when the LED rail is off. 4 x SN74HC595 on VLED (VCC 2-6 V) shift 32 row bits behind the 32 column\nbits; one LAT edge updates rows and columns together. QA..QH drive AO3401A gates (S = VLED, D = ROWn) with 10k\npull-ups to VLED, so rows are off whenever the 595 outputs are Hi-Z. Row pull-downs are DNP options.\n\nScan-stall safety (REQ-L5), CPU-independent: U706 SN74LVC1G123 is retriggered by every MTX_LAT rising edge\n(A low, CLR = MTX_ARM). Q stays high while latches keep arriving. tw: TI guarantees 1.0-1.1 ms at Rext 10k / Cext 0.1 uF (Switching Characteristics 5.8/5.9, VCC 3.3 V,\n-40 to 125 C). Scaling with R (1%) and C709 (X7R +/-10%, +/-15% temperature) as tw ~ R x C gives 0.76-1.41 ms\n(DC bias only shortens it); measure on Rev A.\nThe 1G123 has only a Q output, so U707 inverts it: SAFE = NOT Q (net MTX_SAFE_SENSE, read by P0.21).\nSAFE high (stall, reset, MTX_ARM low) forces BLANK_TLC via U708 and tri-states the 595 outputs (OE_V), so all\nrows and columns turn off. R705 pulls OE_V up to VLED, so the 595s stay off if U701 isolates\n(3V3 gone while VLED is still up). MTX_BLANK pulled up and MTX_ARM pulled down keep the matrix dark with the MCU off.\nResidual: a firmware fault that keeps latching the same row is not caught here (column cap limits current).\nNothing measured."
 		(exclude_from_sim no)
 		(at 50.8 360.68 0)
@@
 				)
 			)
+		)
+	)
+	(symbol
+		(lib_id "Device:R")
+		(at 101.6 139.7 0)
+		(unit 1)
+		(exclude_from_sim no)
+		(in_bom yes)
+		(on_board yes)
+		(dnp no)
+		(property "Reference" "R705"
+			(at 104.14 138.43 0)
+			(effects
+				(font
+					(size 1.27 1.27)
+				)
+				(justify left)
+			)
+		)
+		(property "Value" "100k"
+			(at 104.14 140.97 0)
+			(effects
+				(font
+					(size 1.27 1.27)
+				)
+				(justify left)
+			)
+		)
+		(property "Footprint" "Resistor_SMD:R_0402_1005Metric"
+			(at 101.6 139.7 0)
+			(hide yes)
+			(effects
+				(font
+					(size 1.27 1.27)
+				)
+			)
+		)
+		(property "Datasheet" ""
+			(at 101.6 139.7 0)
+			(hide yes)
+			(effects
+				(font
+					(size 1.27 1.27)
+				)
+			)
+		)
+		(property "Description" "Resistor"
+			(at 101.6 139.7 0)
+			(hide yes)
+			(effects
+				(font
+					(size 1.27 1.27)
+				)
+			)
+		)
+		(property "Manufacturer" "UNI-ROYAL(Uniroyal Elec)"
+			(at 101.6 139.7 0)
+			(hide yes)
+			(effects
+				(font
+					(size 1.27 1.27)
+				)
+			)
+		)
+		(property "MPN" "0402WGF1003TCE"
+			(at 101.6 139.7 0)
+			(hide yes)
+			(effects
+				(font
+					(size 1.27 1.27)
+				)
+			)
+		)
+		(property "LCSC" "C25741"
+			(at 101.6 139.7 0)
+			(hide yes)
+			(effects
+				(font
+					(size 1.27 1.27)
+				)
+			)
+		)
+		(property "Note" "OE_V pull-up: keeps the 595 outputs off (Hi-Z, rows pulled off) when U701 is in VCC isolation (3V3 gone while VLED is still up)"
+			(at 101.6 139.7 0)
+			(hide yes)
+			(effects
+				(font
+					(size 1.27 1.27)
+				)
+			)
+		)
+		(pin "1"
+		)
+		(pin "2"
+		)
+		(instances
+			(project "smart-led-badge"
+				(path "/fefc8d4a-8637-4143-b210-9149e35f9884/81d3bb65-b627-4404-95d7-5959776da8f4"
+					(reference "R705")
+					(unit 1)
+				)
+			)
+		)
+	)
+	(wire
+		(pts
+			(xy 101.6 135.89) (xy 101.6 133.35)
+		)
+		(stroke
+			(width 0)
+			(type default)
+		)
+	)
+	(label "OE_V"
+		(at 101.6 133.35 90)
+		(effects
+			(font
+				(size 1.27 1.27)
+			)
+			(justify left bottom)
+		)
+	)
+	(wire
+		(pts
+			(xy 101.6 143.51) (xy 101.6 146.05)
+		)
+		(stroke
+			(width 0)
+			(type default)
+		)
+	)
+	(global_label "VLED"
+		(shape passive)
+		(at 101.6 146.05 270)
+		(fields_autoplaced yes)
+		(effects
+			(font
+				(size 1.27 1.27)
+			)
+			(justify right)
+		)
+		(property "Intersheetrefs" "${INTERSHEET_REFS}"
+			(at 101.6 146.05 0)
+			(hide yes)
+			(effects
+				(font
+					(size 1.27 1.27)
+				)
+			)
