File: hardware/sheets/usb_charger_battery.kicad_sch (KiCad schematic)
At the start: 43 parts, among them J301 TYPE-C-31-M-12, J302 Battery JST-PH 2P, Q301 AO3400A, Q302 AO3400A, U301 TPD4E05U06, U302 BQ25620

Commit message: hw: use single-sided assembly with a through-hole battery header and low-profile inductors (#11)
* hw: use a through-hole side-entry battery header

The board is assembled on one side only, so the battery header can no
longer be an SMT part on the rear. J302 becomes a JST S2B-PH-K-S
through-hole side-entry header: its body sits on the rear beside the
pack's lead exit and its pins are soldered from the front, outside the
LED field. The footprint matches JST's through-hole layout (circuit 1
position, 2.0 mm pitch, 0.75 mm drill).

The symbol becomes a plain two-pin connector because the part has no
mounting pads. Pin 1 stays BAT- and pin 2 BAT+. An Assembly field marks
the part as hand-soldered after assembly unless the assembler confirms
rear insertion.

* hw: use 2.1 mm XGL4020 inductors for the LED rail and charger

With every part on the front, part height adds directly to the badge
thickness. The 3.1 mm XEL4030 on the LED boost (L202) and charger (L301)
becomes a Coilcraft XGL4020-102MEC, 2.10 mm max, with the same 0.98 x
3.4 mm land pattern at 2.37 mm centres.

The worst-case boost peak is 2.94 A with the 18.0 mA column cap (2.9 V
in, 5.33 V out, 0.66 A, -20 % inductance tolerance, -20 % switching
frequency), below the 3.8 A rating for a 10 % inductance drop. The
earlier 3.66 A figure assumed 35 mA columns. The charger peaks at
2.76 A at the 1.5 A input limit. Current-limit cases stay below the
30 % drop point. These are calculations, not measurements.

* docs: record dual-orientation wear and single-sided assembly

ADR 0009: the badge is worn landscape or portrait, with firmware
rotating the content from the IMU and QR mode keeping its orientation
until it is left. Magnetic and lanyard mounting are both required; the
carrier takes the lanyard load.

ADR 0010: all components are on the front and the rear holds only the
battery, the battery connector body and the carrier. Thickness targets
become regional: about 12 mm over the LED field, 13.5 mm over the
electron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
Parts:
- J302: footprint Connector_JST:JST_PH_B2B-PH-SM4-TB_1x02-1MP_P2.00mm_Vertical -> Connector_JST:JST_PH_S2B-PH-K_1x02_P2.00mm_Horizontal; symbol Connector_Generic_MountingPin:Conn_01x02_MountingPin -> Connector_Generic:Conn_01x02; Assembly (none) -> Hand-solder after PCBA by default (THT, inserted from the r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; LCSC C160352 -> C173752; MPN B2B-PH-SM4-TB(LF)(SN) -> S2B-PH-K-S(LF)(SN); Note Pin 1 = BAT-, pin 2 = BAT+ per Adafruit's own charger desig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 -> Rear side, THT side entry (4.8 mm tall), body beside the pa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
- L301: footprint smart-led-badge:L_Coilcraft_XEL4030 -> smart-led-badge:L_Coilcraft_XGL4020; LCSC C5441341 -> C5357696; MPN XEL4030-102MEC -> XGL4020-102MEC; Note Same part as L202; Isat 9.0 A vs ~2.4 A peak at 1.5 A input -> Same part as L202; Isat 3.8 A (10 % drop) vs 3.0 A calculat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
Connections:
- net GND: no longer J302.MP (MountPin)
Changed lines of the file:
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@@
 	(wire
 		(pts
-			(xy 33.02 172.72) (xy 33.02 175.26)
-		)
-		(stroke
-			(width 0)
-			(type default)
-		)
-	)
-	(wire
-		(pts
 			(xy 167.64 205.74) (xy 167.64 208.28)
 		)
@@
 	)
 	(symbol
-		(lib_id "power:GND")
-		(at 33.02 175.26 0)
-		(unit 1)
-		(body_style 1)
-		(exclude_from_sim no)
-		(in_bom no)
-		(on_board no)
-		(in_pos_files yes)
-		(dnp no)
-		(property "Reference" "#PWR331"
-			(at 33.02 171.45 0)
-			(hide yes)
-			(show_name no)
-			(do_not_autoplace no)
-			(effects
-				(font
-					(size 1.27 1.27)
-				)
-			)
-		)
-		(property "Value" "GND"
-			(at 33.02 179.07 0)
-			(show_name no)
-			(do_not_autoplace no)
-			(effects
-				(font
-					(size 1.27 1.27)
-				)
-			)
-		)
-		(property "Footprint" ""
-			(at 33.02 175.26 0)
-			(hide yes)
-			(show_name no)
-			(do_not_autoplace no)
-			(effects
-				(font
-					(size 1.27 1.27)
-				)
-			)
-		)
-		(property "Datasheet" ""
-			(at 33.02 175.26 0)
-			(hide yes)
-			(show_name no)
-			(do_not_autoplace no)
-			(effects
-				(font
-					(size 1.27 1.27)
-				)
-			)
-		)
-		(property "Description" "Power symbol creates a global label with name \"GND\" , ground"
-			(at 33.02 175.26 0)
-			(hide yes)
-			(show_name no)
-			(do_not_autoplace no)
-			(effects
-				(font
-					(size 1.27 1.27)
-				)
-			)
-		)
-		(pin "1"
-		)
-		(instances
-			(project "smart-led-badge"
-				(path "/fefc8d4a-8637-4143-b210-9149e35f9884/f79dd5bf-1129-4160-8b1f-c78c0c86307a"
-					(reference "#PWR331")
-					(unit 1)
-				)
-			)
-		)
-	)
-	(symbol
 		(lib_id "Device:Thermistor_NTC")
 		(at 320.04 132.08 0)
@@
 			)
 		)
-		(property "Footprint" "smart-led-badge:L_Coilcraft_XEL4030"
+		(property "Footprint" "smart-led-badge:L_Coilcraft_XGL4020"
 			(at 279.4 50.8 0)
 			(hide yes)
@@
 			)
 		)
-		(property "MPN" "XEL4030-102MEC"
+		(property "MPN" "XGL4020-102MEC"
 			(at 279.4 50.8 0)
 			(hide yes)
@@
 			)
 		)
-		(property "LCSC" "C5441341"
+		(property "LCSC" "C5357696"
 			(at 279.4 50.8 0)
 			(hide yes)
@@
 			)
 		)
-		(property "Note" "Same part as L202; Isat 9.0 A vs ~2.4 A peak at 1.5 A input"
+		(property "Note" "Same part as L202; Isat 3.8 A (10 % drop) vs 3.0 A calculated peak at IINDPM 1.5 A (efficiency 100 %, 1.35 MHz); measure at bring-up"
 			(at 279.4 50.8 0)
 			(hide yes)
@@
 	)
 	(symbol
-		(lib_id "Connector_Generic_MountingPin:Conn_01x02_MountingPin")
+		(lib_id "Connector_Generic:Conn_01x02")
 		(at 33.02 165.1 0)
 		(unit 1)
@@
 			)
 		)
-		(property "Footprint" "Connector_JST:JST_PH_B2B-PH-SM4-TB_1x02-1MP_P2.00mm_Vertical"
+		(property "Footprint" "Connector_JST:JST_PH_S2B-PH-K_1x02_P2.00mm_Horizontal"
 			(at 33.02 165.1 0)
 			(hide yes)
@@
 			)
 		)
-		(property "Description" "Generic connectable mounting pin connector, single row, 01x02, script generated (kicad-library-utils/schlib/autogen/connector/)"
+		(property "Description" "Generic connector, single row, 01x02, script generated (kicad-library-utils/schlib/autogen/connector/)"
 			(at 33.02 165.1 0)
 			(hide yes)
@@
 			)
 		)
-		(property "MPN" "B2B-PH-SM4-TB(LF)(SN)"
+		(property "Assembly" "Hand-solder after PCBA by default (THT, inserted from the rear, soldered from the front); assembler only if it confirms rear insertion"
 			(at 33.02 165.1 0)
 			(hide yes)
@@
 			)
 		)
-		(property "LCSC" "C160352"
+		(property "MPN" "S2B-PH-K-S(LF)(SN)"
 			(at 33.02 165.1 0)
 			(hide yes)
@@
 			)
 		)
-		(property "Note" "Pin 1 = BAT-, pin 2 = BAT+ per Adafruit's own charger design (Micro-Lipo USB-C CN2: pin 1 GND, pin 2 VBAT) and Adafruit's statement that product 328 matches its boards; meter-check the pack before first connection"
+		(property "LCSC" "C173752"
+			(at 33.02 165.1 0)
+			(hide yes)
+			(show_name no)
+			(do_not_autoplace no)
+			(effects
+				(font
+					(size 1.27 1.27)
+				)
+			)
+		)
+		(property "Note" "Rear side, THT side entry (4.8 mm tall), body beside the pack, soldered from the front outside the LED field; the only rear part besides the battery. Pin 1 = BAT-, pin 2 = BAT+ per Adafruit's own charger design (Micro-Lipo USB-C CN2: pin 1 GND, pin 2 VBAT) and Adafruit's statement that product 328 matches its boards; meter-check the pack before first connection"
 			(at 33.02 165.1 0)
 			(hide yes)
@@
 		(pin "2"
 		)
-		(pin "MP"
-		)
 		(instances
