File: hardware/sheets/user_interface.kicad_sch (KiCad schematic)
At the start: 0 parts

Commit message: hw: draw UI, IMU, microphone and NFC sheets
IMU: ICM-42688-P on the shared I2C1 bus at 0x68, bypassed as TDK's
application circuit specifies, reserved pins to ground, and unfitted
links for the SPI fallback.

Microphone: SPH0641LM4H-1 with a C0G bypass capacitor (Knowles advises
against class 2 dielectrics next to the part), a 0 ohm supply link for
current measurement, series options on clock and data, and SELECT to
ground.

NFC: NT3H2111W0FHKH powered from the NFC_PWR GPIO with its bus and
field-detect pull-ups, the PCB coil as a non-BOM part, two unfitted
tuning capacitor positions and test points for bus timing.

UI: two tact switches to ground with unfitted external pull-ups and a
red status LED.

The labels these sheets connect no longer need ERC exclusions. NFC_PWR
gets a reviewed exclusion: a GPIO drives the tag supply by design.
Parts:
- added D1201: Red, LED_SMD:LED_0603_1608Metric, symbol Device:LED
- added R1201, R1202: 10k, Resistor_SMD:R_0402_1005Metric, symbol Device:R
- added R1203: 1k, Resistor_SMD:R_0402_1005Metric, symbol Device:R
- added SW1201: Mode/Next, smart-led-badge:SW_XUNPU_TS-1088, symbol Switch:SW_Push
- added SW1202: Action/Select, smart-led-badge:SW_XUNPU_TS-1088, symbol Switch:SW_Push
Connections:
- new net +3V3: R1201.2, R1202.2
- new net BTN_ACTION: R1202.1, SW1202.1
- new net BTN_MODE: R1201.1, SW1201.1
- new net GND: D1201.1 (K), SW1201.2, SW1202.2
- new net LED_A: D1201.2 (A), R1203.2
- new net STATUS_LED: R1203.1
Other:
- note added: "User interface (Rev A) - design notes Two buttons (Mode/Next, Action/Select; long press allowed) to GND, internal pull-ups; DNP external pull-ups. Placement (OD-27): front face in the strip below the LED field if the land pattern fits with LED and edge clearance; otherwise side-actuated parts on the bottom edge. Contacts are enclosed under a plastic actuator. Status LED on the rear, GPIO high = o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"
