File: hardware/sheets/led_matrix.kicad_sch (KiCad schematic)
At the start: 1024 parts

Commit message: hw: apply layout footprint and test-point changes to the schematic
The matrix LEDs use the KENTO-pattern footprint, L1101 the PCB coil,
MK1001 the 0.6 mm hole footprint and J301 the project HRO copy.

Removes test points that duplicate others: TP303 and TP304, TP208 and
TP506, and TP501-TP503, whose signals are on the SWD header. Also
removes H1304, which the carrier does not use. Rail and GND test points
move to 0.8 mm pads.

nRESET now connects only the header's open-collector pin and the module
input. ERC reports that as not driven, so the error is excluded: the
nRF5340 has an internal pull-up on reset.
Parts:
- LD1000, LD1001, LD1002, LD1003, LD1004, LD1005, LD1006, LD1007, LD1008, LD1009, LD1010, LD1011, LD1012, LD1013, LD1014, LD1015, LD1016, LD1017, LD1018, LD1019, LD1020, LD1021, LD1022, LD1023, LD1024, LD1025, LD1026, LD1027, LD1028, LD1029, LD1030, LD1031, LD1100, LD1101, LD1102, LD1103, LD1104, LD1105, LD1106, LD1107, LD1108, LD1109, LD1110, LD1111, LD1112, LD1113, LD1114, LD1115, LD1116, LD1117, LD1118, LD1119, LD1120, LD1121, LD1122, LD1123, LD1124, LD1125, LD1126, LD1127, LD1128, LD1129, LD1130, LD1131, LD1200, LD1201, LD1202, LD1203, LD1204, LD1205, LD1206, LD1207, LD1208, LD1209, LD1210, LD1211, LD1212, LD1213, LD1214, LD1215, LD1216, LD1217, LD1218, LD1219, LD1220, LD1221, LD1222, LD1223, LD1224, LD1225, LD1226, LD1227, LD1228, LD1229, LD1230, LD1231, LD1300, LD1301, LD1302, LD1303, LD1304, LD1305, LD1306, LD1307, LD1308, LD1309, LD1310, LD1311, LD1312, LD1313, LD1314, LD1315, LD1316, LD1317, LD1318, LD1319, LD1320, LD1321, LD1322, LD1323, LD1324, LD1325, LD1326, LD1327, LD1328, LD1329, LD1330, LD1331, LD1400, LD1401, LD1402, LD1403, LD1404, LD1405, LD1406, LD1407, LD1408, LD1409, LD1410, LD1411, LD1412, LD1413, LD1414, LD1415, LD1416, LD1417, LD1418, LD1419, LD1420, LD1421, LD1422, LD1423, LD1424, LD1425, LD1426, LD1427, LD1428, LD1429, LD1430, LD1431, LD1500, LD1501, LD1502, LD1503, LD1504, LD1505, LD1506, LD1507, LD1508, LD1509, LD1510, LD1511, LD1512, LD1513, LD1514, LD1515, LD1516, LD1517, LD1518, LD1519, LD1520, LD1521, LD1522, LD1523, LD1524, LD1525, LD1526, LD1527, LD1528, LD1529, LD1530, LD1531, LD1600, LD1601, LD1602, LD1603, LD1604, LD1605, LD1606, LD1607, LD1608, LD1609, LD1610, LD1611, LD1612, LD1613, LD1614, LD1615, LD1616, LD1617, LD1618, LD1619, LD1620, LD1621, LD1622, LD1623, LD1624, LD1625, LD1626, LD1627, LD1628, LD1629, LD1630, LD1631, LD1700, LD1701, LD1702, LD1703, LD1704, LD1705, LD1706, LD1707, LD1708, LD1709, LD1710, LD1711, LD1712, LD1713, LD1714, LD1715, LD1716, LD1717, LD1718, LD1719, LD1720, LD1721, LD1722, LD1723, LD1724, LD1725, LD1726, LD1727, LD1728, LD1729, LD1730, LD1731, LD1800, LD1801, LD1802, LD1803, LD1804, LD1805, LD1806, LD1807, LD1808, LD1809, LD1810, LD1811, LD1812, LD1813, LD1814, LD1815, LD1816, LD1817, LD1818, LD1819, LD1820, LD1821, LD1822, LD1823, LD1824, LD1825, LD1826, LD1827, LD1828, LD1829, LD1830, LD1831, LD1900, LD1901, LD1902, LD1903, LD1904, LD1905, LD1906, LD1907, LD1908, LD1909, LD1910, LD1911, LD1912, LD1913, LD1914, LD1915, LD1916, LD1917, LD1918, LD1919, LD1920, LD1921, LD1922, LD1923, LD1924, LD1925, LD1926, LD1927, LD1928, LD1929, LD1930, LD1931, LD2000, LD2001, LD2002, LD2003, LD2004, LD2005, LD2006, LD2007, LD2008, LD2009, LD2010, LD2011, LD2012, LD2013, LD2014, LD2015, LD2016, LD2017, LD2018, LD2019, LD2020, LD2021, LD2022, LD2023, LD2024, LD2025, LD2026, LD2027, LD2028, LD2029, LD2030, LD2031, LD2100, LD2101, LD2102, LD2103, LD2104, LD2105, LD2106, LD2107, LD2108, LD2109, LD2110, LD2111, LD2112, LD2113, LD2114, LD2115, LD2116, LD2117, LD2118, LD2119, LD2120, LD2121, LD2122, LD2123, LD2124, LD2125, LD2126, LD2127, LD2128, LD2129, LD2130, LD2131, LD2200, LD2201, LD2202, LD2203, LD2204, LD2205, LD2206, LD2207, LD2208, LD2209, LD2210, LD2211, LD2212, LD2213, LD2214, LD2215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: footprint LED_SMD:LED_0603_1608Metric -> smart-led-badge:LED_0603_KENTO_KT-0603

Commit message: hw: select the KT-0603W as the matrix LED
The ratings in KENTO's datasheet cover the matrix drive. The 18-19.4 mA
peak at 1/32 duty is below the 30 mA DC rating. A row held on by a fault
stays within the DC and 100 mW limits at badge ambient.

Worst-case forward voltage needs a VLED of about 4.34 V, against 4.75 V
nominal. Reverse bias in the matrix stays near 2.5 V, well under the
5 V limit.

Brightness and bin uniformity could not be compared on samples, so they
are measured on Rev A along with QR scanning. The LED notes in the
schematic and on the board, the hardware status and the references now
show the part as selected.
Parts:
- LD1000, LD1001, LD1002, LD1003, LD1004, LD1005, LD1006, LD1007, LD1008, LD1009, LD1010, LD1011, LD1012, LD1013, LD1014, LD1015, LD1016, LD1017, LD1018, LD1019, LD1020, LD1021, LD1022, LD1023, LD1024, LD1025, LD1026, LD1027, LD1028, LD1029, LD1030, LD1031, LD1100, LD1101, LD1102, LD1103, LD1104, LD1105, LD1106, LD1107, LD1108, LD1109, LD1110, LD1111, LD1112, LD1113, LD1114, LD1115, LD1116, LD1117, LD1118, LD1119, LD1120, LD1121, LD1122, LD1123, LD1124, LD1125, LD1126, LD1127, LD1128, LD1129, LD1130, LD1131, LD1200, LD1201, LD1202, LD1203, LD1204, LD1205, LD1206, LD1207, LD1208, LD1209, LD1210, LD1211, LD1212, LD1213, LD1214, LD1215, LD1216, LD1217, LD1218, LD1219, LD1220, LD1221, LD1222, LD1223, LD1224, LD1225, LD1226, LD1227, LD1228, LD1229, LD1230, LD1231, LD1300, LD1301, LD1302, LD1303, LD1304, LD1305, LD1306, LD1307, LD1308, LD1309, LD1310, LD1311, LD1312, LD1313, LD1314, LD1315, LD1316, LD1317, LD1318, LD1319, LD1320, LD1321, LD1322, LD1323, LD1324, LD1325, LD1326, LD1327, LD1328, LD1329, LD1330, LD1331, LD1400, LD1401, LD1402, LD1403, LD1404, LD1405, LD1406, LD1407, LD1408, LD1409, LD1410, LD1411, LD1412, LD1413, LD1414, LD1415, LD1416, LD1417, LD1418, LD1419, LD1420, LD1421, LD1422, LD1423, LD1424, LD1425, LD1426, LD1427, LD1428, LD1429, LD1430, LD1431, LD1500, LD1501, LD1502, LD1503, LD1504, LD1505, LD1506, LD1507, LD1508, LD1509, LD1510, LD1511, LD1512, LD1513, LD1514, LD1515, LD1516, LD1517, LD1518, LD1519, LD1520, LD1521, LD1522, LD1523, LD1524, LD1525, LD1526, LD1527, LD1528, LD1529, LD1530, LD1531, LD1600, LD1601, LD1602, LD1603, LD1604, LD1605, LD1606, LD1607, LD1608, LD1609, LD1610, LD1611, LD1612, LD1613, LD1614, LD1615, LD1616, LD1617, LD1618, LD1619, LD1620, LD1621, LD1622, LD1623, LD1624, LD1625, LD1626, LD1627, LD1628, LD1629, LD1630, LD1631, LD1700, LD1701, LD1702, LD1703, LD1704, LD1705, LD1706, LD1707, LD1708, LD1709, LD1710, LD1711, LD1712, LD1713, LD1714, LD1715, LD1716, LD1717, LD1718, LD1719, LD1720, LD1721, LD1722, LD1723, LD1724, LD1725, LD1726, LD1727, LD1728, LD1729, LD1730, LD1731, LD1800, LD1801, LD1802, LD1803, LD1804, LD1805, LD1806, LD1807, LD1808, LD1809, LD1810, LD1811, LD1812, LD1813, LD1814, LD1815, LD1816, LD1817, LD1818, LD1819, LD1820, LD1821, LD1822, LD1823, LD1824, LD1825, LD1826, LD1827, LD1828, LD1829, LD1830, LD1831, LD1900, LD1901, LD1902, LD1903, LD1904, LD1905, LD1906, LD1907, LD1908, LD1909, LD1910, LD1911, LD1912, LD1913, LD1914, LD1915, LD1916, LD1917, LD1918, LD1919, LD1920, LD1921, LD1922, LD1923, LD1924, LD1925, LD1926, LD1927, LD1928, LD1929, LD1930, LD1931, LD2000, LD2001, LD2002, LD2003, LD2004, LD2005, LD2006, LD2007, LD2008, LD2009, LD2010, LD2011, LD2012, LD2013, LD2014, LD2015, LD2016, LD2017, LD2018, LD2019, LD2020, LD2021, LD2022, LD2023, LD2024, LD2025, LD2026, LD2027, LD2028, LD2029, LD2030, LD2031, LD2100, LD2101, LD2102, LD2103, LD2104, LD2105, LD2106, LD2107, LD2108, LD2109, LD2110, LD2111, LD2112, LD2113, LD2114, LD2115, LD2116, LD2117, LD2118, LD2119, LD2120, LD2121, LD2122, LD2123, LD2124, LD2125, LD2126, LD2127, LD2128, LD2129, LD2130, LD2131, LD2200, LD2201, LD2202, LD2203, LD2204, LD2205, LD2206, LD2207, LD2208, LD2209, LD2210, LD2211, LD2212, LD2213, LD2214, LD2215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: Note Matrix LED PROTOTYPE-DEPENDENT (OD-03); front side, 2.0 mm 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 -> Matrix LED, selected on the KENTO datasheet (2026-10-08); f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
