File: hardware/sheets/led_matrix.kicad_sch (KiCad schematic)
At the start: 0 parts

Commit message: hw: draw LED matrix, row and column drivers and scan-stall safety (#8)
* repo: ignore KiCad local history

KiCad 10 keeps automatic snapshots in a .history folder (with its own
Git repository) next to the project. Ignore it, and make the hygiene
check reject it, so local history cannot be committed.

* hw: save schematic sheets in KiCad's own format

Opening and saving the project in KiCad 10 rewrites the generated
sheets and project file in its native layout. KiCad also merges seven
overlapping wire segments on the USB sheet. Nets, values and
footprints are unchanged, so committing this once keeps later edits
made in KiCad free of formatting churn.

* hw: add column driver and monostable symbols

Add a TLC59283 symbol with the RGE (VQFN-24) pin numbers from TI's pin
table; it uses KiCad's footprint for TI's RGE0024C package. Add a
single-unit SN74LVC1G123 symbol, because KiCad's version keeps the
supply pins in a separate unit.

* hw: draw matrix driver and LED matrix sheets

Columns: two cascaded TLC59283 sinks on 3V3. R_IREF is 2.94k, an
18.0 mA nominal setting (about 19.4 mA worst case with driver and
resistor tolerance), with a fitted 0 ohm in series, so adjustment can
only lower the current.

Rows: the TLC chain output, clock, latch and SAFE cross into the LED
rail through an SN74LVC8T245 translator. Four SN74HC595 on VLED drive
32 AO3401A high-side switches with 10k gate pull-ups, with row
pull-downs as unfitted options.

Scan-stall safety: every latch retriggers an SN74LVC1G123. TI
specifies 1.0-1.1 ms at 10k / 0.1 uF; with the fitted parts'
tolerances the timeout is 0.76-1.41 ms. The part has only a Q
output, so an inverter makes SAFE = NOT Q. SAFE forces the column
BLANK through an OR gate and tri-states the row registers, and the
MCU reads it. The matrix stays dark while the MCU is off or in
reset.

LED matrix: 1024 LEDs, anodes on the rows and cathodes on the
columns, drawn as row and column buses, on the front side with the
buttons (ADR 0008).

The pend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
Parts:
- added LD1000, LD1001, LD1002, LD1003, LD1004, LD1005, LD1006, LD1007, LD1008, LD1009, LD1010, LD1011, LD1012, LD1013, LD1014, LD1015, LD1016, LD1017, LD1018, LD1019, LD1020, LD1021, LD1022, LD1023, LD1024, LD1025, LD1026, LD1027, LD1028, LD1029, LD1030, LD1031, LD1100, LD1101, LD1102, LD1103, LD1104, LD1105, LD1106, LD1107, LD1108, LD1109, LD1110, LD1111, LD1112, LD1113, LD1114, LD1115, LD1116, LD1117, LD1118, LD1119, LD1120, LD1121, LD1122, LD1123, LD1124, LD1125, LD1126, LD1127, LD1128, LD1129, LD1130, LD1131, LD1200, LD1201, LD1202, LD1203, LD1204, LD1205, LD1206, LD1207, LD1208, LD1209, LD1210, LD1211, LD1212, LD1213, LD1214, LD1215, LD1216, LD1217, LD1218, LD1219, LD1220, LD1221, LD1222, LD1223, LD1224, LD1225, LD1226, LD1227, LD1228, LD1229, LD1230, LD1231, LD1300, LD1301, LD1302, LD1303, LD1304, LD1305, LD1306, LD1307, LD1308, LD1309, LD1310, LD1311, LD1312, LD1313, LD1314, LD1315, LD1316, LD1317, LD1318, LD1319, LD1320, LD1321, LD1322, LD1323, LD1324, LD1325, LD1326, LD1327, LD1328, LD1329, LD1330, LD1331, LD1400, LD1401, LD1402, LD1403, LD1404, LD1405, LD1406, LD1407, LD1408, LD1409, LD1410, LD1411, LD1412, LD1413, LD1414, LD1415, LD1416, LD1417, LD1418, LD1419, LD1420, LD1421, LD1422, LD1423, LD1424, LD1425, LD1426, LD1427, LD1428, LD1429, LD1430, LD1431, LD1500, LD1501, LD1502, LD1503, LD1504, LD1505, LD1506, LD1507, LD1508, LD1509, LD1510, LD1511, LD1512, LD1513, LD1514, LD1515, LD1516, LD1517, LD1518, LD1519, LD1520, LD1521, LD1522, LD1523, LD1524, LD1525, LD1526, LD1527, LD1528, LD1529, LD1530, LD1531, LD1600, LD1601, LD1602, LD1603, LD1604, LD1605, LD1606, LD1607, LD1608, LD1609, LD1610, LD1611, LD1612, LD1613, LD1614, LD1615, LD1616, LD1617, LD1618, LD1619, LD1620, LD1621, LD1622, LD1623, LD1624, LD1625, LD1626, LD1627, LD1628, LD1629, LD1630, LD1631, LD1700, LD1701, LD1702, LD1703, LD1704, LD1705, LD1706, LD1707, LD1708, LD1709, LD1710, LD1711, LD1712, LD1713, LD1714, LD1715, LD1716, LD1717, LD1718, LD1719, LD1720, LD1721, LD1722, LD1723, LD1724, LD1725, LD1726, LD1727, LD1728, LD1729, LD1730, LD1731, LD1800, LD1801, LD1802, LD1803, LD1804, LD1805, LD1806, LD1807, LD1808, LD1809, LD1810, LD1811, LD1812, LD1813, LD1814, LD1815, LD1816, LD1817, LD1818, LD1819, LD1820, LD1821, LD1822, LD1823, LD1824, LD1825, LD1826, LD1827, LD1828, LD1829, LD1830, LD1831, LD1900, LD1901, LD1902, LD1903, LD1904, LD1905, LD1906, LD1907, LD1908, LD1909, LD1910, LD1911, LD1912, LD1913, LD1914, LD1915, LD1916, LD1917, LD1918, LD1919, LD1920, LD1921, LD1922, LD1923, LD1924, LD1925, LD1926, LD1927, LD1928, LD1929, LD1930, LD1931, LD2000, LD2001, LD2002, LD2003, LD2004, LD2005, LD2006, LD2007, LD2008, LD2009, LD2010, LD2011, LD2012, LD2013, LD2014, LD2015, LD2016, LD2017, LD2018, LD2019, LD2020, LD2021, LD2022, LD2023, LD2024, LD2025, LD2026, LD2027, LD2028, LD2029, LD2030, LD2031, LD2100, LD2101, LD2102, LD2103, LD2104, LD2105, LD2106, LD2107, LD2108, LD2109, LD2110, LD2111, LD2112, LD2113, LD2114, LD2115, LD2116, LD2117, LD2118, LD2119, LD2120, LD2121, LD2122, LD2123, LD2124, LD2125, LD2126, LD2127, LD2128, LD2129, LD2130, LD2131, LD2200, LD2201, LD2202, LD2203, LD2204, LD2205, LD2206, LD2207, LD2208, LD2209, LD2210, LD2211, LD2212, LD2213, LD2214, LD2215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: KT-0603W, LED_SMD:LED_0603_1608Metric, symbol Device:LED
Connections:
- new net COL0: LD1000.1 (K), LD1100.1 (K), LD1200.1 (K), LD1300.1 (K), LD1400.1 (K), LD1500.1 (K), LD1600.1 (K), LD1700.1 (K), LD1800.1 (K), LD1900.1 (K), LD2000.1 (K), LD2100.1 (K), LD2200.1 (K), LD2300.1 (K), LD2400.1 (K), LD2500.1 (K), LD2600.1 (K), LD2700.1 (K), LD2800.1 (K), LD2900.1 (K), LD3000.1 (K), LD3100.1 (K), LD3200.1 (K), LD3300.1 (K), LD3400.1 (K), LD3500.1 (K), LD3600.1 (K), LD3700.1 (K), LD3800.1 (K), LD3900.1 (K), LD4000.1 (K), LD4100.1 (K)
- new net COL1: LD1001.1 (K), LD1101.1 (K), LD1201.1 (K), LD1301.1 (K), LD1401.1 (K), LD1501.1 (K), LD1601.1 (K), LD1701.1 (K), LD1801.1 (K), LD1901.1 (K), LD2001.1 (K), LD2101.1 (K), LD2201.1 (K), LD2301.1 (K), LD2401.1 (K), LD2501.1 (K), LD2601.1 (K), LD2701.1 (K), LD2801.1 (K), LD2901.1 (K), LD3001.1 (K), LD3101.1 (K), LD3201.1 (K), LD3301.1 (K), LD3401.1 (K), LD3501.1 (K), LD3601.1 (K), LD3701.1 (K), LD3801.1 (K), LD3901.1 (K), LD4001.1 (K), LD4101.1 (K)
- new net COL10: LD1010.1 (K), LD1110.1 (K), LD1210.1 (K), LD1310.1 (K), LD1410.1 (K), LD1510.1 (K), LD1610.1 (K), LD1710.1 (K), LD1810.1 (K), LD1910.1 (K), LD2010.1 (K), LD2110.1 (K), LD2210.1 (K), LD2310.1 (K), LD2410.1 (K), LD2510.1 (K), LD2610.1 (K), LD2710.1 (K), LD2810.1 (K), LD2910.1 (K), LD3010.1 (K), LD3110.1 (K), LD3210.1 (K), LD3310.1 (K), LD3410.1 (K), LD3510.1 (K), LD3610.1 (K), LD3710.1 (K), LD3810.1 (K), LD3910.1 (K), LD4010.1 (K), LD4110.1 (K)
- new net COL11: LD1011.1 (K), LD1111.1 (K), LD1211.1 (K), LD1311.1 (K), LD1411.1 (K), LD1511.1 (K), LD1611.1 (K), LD1711.1 (K), LD1811.1 (K), LD1911.1 (K), LD2011.1 (K), LD2111.1 (K), LD2211.1 (K), LD2311.1 (K), LD2411.1 (K), LD2511.1 (K), LD2611.1 (K), LD2711.1 (K), LD2811.1 (K), LD2911.1 (K), LD3011.1 (K), LD3111.1 (K), LD3211.1 (K), LD3311.1 (K), LD3411.1 (K), LD3511.1 (K), LD3611.1 (K), LD3711.1 (K), LD3811.1 (K), LD3911.1 (K), LD4011.1 (K), LD4111.1 (K)
- new net COL12: LD1012.1 (K), LD1112.1 (K), LD1212.1 (K), LD1312.1 (K), LD1412.1 (K), LD1512.1 (K), LD1612.1 (K), LD1712.1 (K), LD1812.1 (K), LD1912.1 (K), LD2012.1 (K), LD2112.1 (K), LD2212.1 (K), LD2312.1 (K), LD2412.1 (K), LD2512.1 (K), LD2612.1 (K), LD2712.1 (K), LD2812.1 (K), LD2912.1 (K), LD3012.1 (K), LD3112.1 (K), LD3212.1 (K), LD3312.1 (K), LD3412.1 (K), LD3512.1 (K), LD3612.1 (K), LD3712.1 (K), LD3812.1 (K), LD3912.1 (K), LD4012.1 (K), LD4112.1 (K)
- new net COL13: LD1013.1 (K), LD1113.1 (K), LD1213.1 (K), LD1313.1 (K), LD1413.1 (K), LD1513.1 (K), LD1613.1 (K), LD1713.1 (K), LD1813.1 (K), LD1913.1 (K), LD2013.1 (K), LD2113.1 (K), LD2213.1 (K), LD2313.1 (K), LD2413.1 (K), LD2513.1 (K), LD2613.1 (K), LD2713.1 (K), LD2813.1 (K), LD2913.1 (K), LD3013.1 (K), LD3113.1 (K), LD3213.1 (K), LD3313.1 (K), LD3413.1 (K), LD3513.1 (K), LD3613.1 (K), LD3713.1 (K), LD3813.1 (K), LD3913.1 (K), LD4013.1 (K), LD4113.1 (K)
- new net COL14: LD1014.1 (K), LD1114.1 (K), LD1214.1 (K), LD1314.1 (K), LD1414.1 (K), LD1514.1 (K), LD1614.1 (K), LD1714.1 (K), LD1814.1 (K), LD1914.1 (K), LD2014.1 (K), LD2114.1 (K), LD2214.1 (K), LD2314.1 (K), LD2414.1 (K), LD2514.1 (K), LD2614.1 (K), LD2714.1 (K), LD2814.1 (K), LD2914.1 (K), LD3014.1 (K), LD3114.1 (K), LD3214.1 (K), LD3314.1 (K), LD3414.1 (K), LD3514.1 (K), LD3614.1 (K), LD3714.1 (K), LD3814.1 (K), LD3914.1 (K), LD4014.1 (K), LD4114.1 (K)
- new net COL15: LD1015.1 (K), LD1115.1 (K), LD1215.1 (K), LD1315.1 (K), LD1415.1 (K), LD1515.1 (K), LD1615.1 (K), LD1715.1 (K), LD1815.1 (K), LD1915.1 (K), LD2015.1 (K), LD2115.1 (K), LD2215.1 (K), LD2315.1 (K), LD2415.1 (K), LD2515.1 (K), LD2615.1 (K), LD2715.1 (K), LD2815.1 (K), LD2915.1 (K), LD3015.1 (K), LD3115.1 (K), LD3215.1 (K), LD3315.1 (K), LD3415.1 (K), LD3515.1 (K), LD3615.1 (K), LD3715.1 (K), LD3815.1 (K), LD3915.1 (K), LD4015.1 (K), LD4115.1 (K)
- new net COL16: LD1016.1 (K), LD1116.1 (K), LD1216.1 (K), LD1316.1 (K), LD1416.1 (K), LD1516.1 (K), LD1616.1 (K), LD1716.1 (K), LD1816.1 (K), LD1916.1 (K), LD2016.1 (K), LD2116.1 (K), LD2216.1 (K), LD2316.1 (K), LD2416.1 (K), LD2516.1 (K), LD2616.1 (K), LD2716.1 (K), LD2816.1 (K), LD2916.1 (K), LD3016.1 (K), LD3116.1 (K), LD3216.1 (K), LD3316.1 (K), LD3416.1 (K), LD3516.1 (K), LD3616.1 (K), LD3716.1 (K), LD3816.1 (K), LD3916.1 (K), LD4016.1 (K), LD4116.1 (K)
- new net COL17: LD1017.1 (K), LD1117.1 (K), LD1217.1 (K), LD1317.1 (K), LD1417.1 (K), LD1517.1 (K), LD1617.1 (K), LD1717.1 (K), LD1817.1 (K), LD1917.1 (K), LD2017.1 (K), LD2117.1 (K), LD2217.1 (K), LD2317.1 (K), LD2417.1 (K), LD2517.1 (K), LD2617.1 (K), LD2717.1 (K), LD2817.1 (K), LD2917.1 (K), LD3017.1 (K), LD3117.1 (K), LD3217.1 (K), LD3317.1 (K), LD3417.1 (K), LD3517.1 (K), LD3617.1 (K), LD3717.1 (K), LD3817.1 (K), LD3917.1 (K), LD4017.1 (K), LD4117.1 (K)
- new net COL18: LD1018.1 (K), LD1118.1 (K), LD1218.1 (K), LD1318.1 (K), LD1418.1 (K), LD1518.1 (K), LD1618.1 (K), LD1718.1 (K), LD1818.1 (K), LD1918.1 (K), LD2018.1 (K), LD2118.1 (K), LD2218.1 (K), LD2318.1 (K), LD2418.1 (K), LD2518.1 (K), LD2618.1 (K), LD2718.1 (K), LD2818.1 (K), LD2918.1 (K), LD3018.1 (K), LD3118.1 (K), LD3218.1 (K), LD3318.1 (K), LD3418.1 (K), LD3518.1 (K), LD3618.1 (K), LD3718.1 (K), LD3818.1 (K), LD3918.1 (K), LD4018.1 (K), LD4118.1 (K)
- new net COL19: LD1019.1 (K), LD1119.1 (K), LD1219.1 (K), LD1319.1 (K), LD1419.1 (K), LD1519.1 (K), LD1619.1 (K), LD1719.1 (K), LD1819.1 (K), LD1919.1 (K), LD2019.1 (K), LD2119.1 (K), LD2219.1 (K), LD2319.1 (K), LD2419.1 (K), LD2519.1 (K), LD2619.1 (K), LD2719.1 (K), LD2819.1 (K), LD2919.1 (K), LD3019.1 (K), LD3119.1 (K), LD3219.1 (K), LD3319.1 (K), LD3419.1 (K), LD3519.1 (K), LD3619.1 (K), LD3719.1 (K), LD3819.1 (K), LD3919.1 (K), LD4019.1 (K), LD4119.1 (K)
- new net COL2: LD1002.1 (K), LD1102.1 (K), LD1202.1 (K), LD1302.1 (K), LD1402.1 (K), LD1502.1 (K), LD1602.1 (K), LD1702.1 (K), LD1802.1 (K), LD1902.1 (K), LD2002.1 (K), LD2102.1 (K), LD2202.1 (K), LD2302.1 (K), LD2402.1 (K), LD2502.1 (K), LD2602.1 (K), LD2702.1 (K), LD2802.1 (K), LD2902.1 (K), LD3002.1 (K), LD3102.1 (K), LD3202.1 (K), LD3302.1 (K), LD3402.1 (K), LD3502.1 (K), LD3602.1 (K), LD3702.1 (K), LD3802.1 (K), LD3902.1 (K), LD4002.1 (K), LD4102.1 (K)
- new net COL20: LD1020.1 (K), LD1120.1 (K), LD1220.1 (K), LD1320.1 (K), LD1420.1 (K), LD1520.1 (K), LD1620.1 (K), LD1720.1 (K), LD1820.1 (K), LD1920.1 (K), LD2020.1 (K), LD2120.1 (K), LD2220.1 (K), LD2320.1 (K), LD2420.1 (K), LD2520.1 (K), LD2620.1 (K), LD2720.1 (K), LD2820.1 (K), LD2920.1 (K), LD3020.1 (K), LD3120.1 (K), LD3220.1 (K), LD3320.1 (K), LD3420.1 (K), LD3520.1 (K), LD3620.1 (K), LD3720.1 (K), LD3820.1 (K), LD3920.1 (K), LD4020.1 (K), LD4120.1 (K)
- new net COL21: LD1021.1 (K), LD1121.1 (K), LD1221.1 (K), LD1321.1 (K), LD1421.1 (K), LD1521.1 (K), LD1621.1 (K), LD1721.1 (K), LD1821.1 (K), LD1921.1 (K), LD2021.1 (K), LD2121.1 (K), LD2221.1 (K), LD2321.1 (K), LD2421.1 (K), LD2521.1 (K), LD2621.1 (K), LD2721.1 (K), LD2821.1 (K), LD2921.1 (K), LD3021.1 (K), LD3121.1 (K), LD3221.1 (K), LD3321.1 (K), LD3421.1 (K), LD3521.1 (K), LD3621.1 (K), LD3721.1 (K), LD3821.1 (K), LD3921.1 (K), LD4021.1 (K), LD4121.1 (K)
- new net COL22: LD1022.1 (K), LD1122.1 (K), LD1222.1 (K), LD1322.1 (K), LD1422.1 (K), LD1522.1 (K), LD1622.1 (K), LD1722.1 (K), LD1822.1 (K), LD1922.1 (K), LD2022.1 (K), LD2122.1 (K), LD2222.1 (K), LD2322.1 (K), LD2422.1 (K), LD2522.1 (K), LD2622.1 (K), LD2722.1 (K), LD2822.1 (K), LD2922.1 (K), LD3022.1 (K), LD3122.1 (K), LD3222.1 (K), LD3322.1 (K), LD3422.1 (K), LD3522.1 (K), LD3622.1 (K), LD3722.1 (K), LD3822.1 (K), LD3922.1 (K), LD4022.1 (K), LD4122.1 (K)
- new net COL23: LD1023.1 (K), LD1123.1 (K), LD1223.1 (K), LD1323.1 (K), LD1423.1 (K), LD1523.1 (K), LD1623.1 (K), LD1723.1 (K), LD1823.1 (K), LD1923.1 (K), LD2023.1 (K), LD2123.1 (K), LD2223.1 (K), LD2323.1 (K), LD2423.1 (K), LD2523.1 (K), LD2623.1 (K), LD2723.1 (K), LD2823.1 (K), LD2923.1 (K), LD3023.1 (K), LD3123.1 (K), LD3223.1 (K), LD3323.1 (K), LD3423.1 (K), LD3523.1 (K), LD3623.1 (K), LD3723.1 (K), LD3823.1 (K), LD3923.1 (K), LD4023.1 (K), LD4123.1 (K)
- new net COL24: LD1024.1 (K), LD1124.1 (K), LD1224.1 (K), LD1324.1 (K), LD1424.1 (K), LD1524.1 (K), LD1624.1 (K), LD1724.1 (K), LD1824.1 (K), LD1924.1 (K), LD2024.1 (K), LD2124.1 (K), LD2224.1 (K), LD2324.1 (K), LD2424.1 (K), LD2524.1 (K), LD2624.1 (K), LD2724.1 (K), LD2824.1 (K), LD2924.1 (K), LD3024.1 (K), LD3124.1 (K), LD3224.1 (K), LD3324.1 (K), LD3424.1 (K), LD3524.1 (K), LD3624.1 (K), LD3724.1 (K), LD3824.1 (K), LD3924.1 (K), LD4024.1 (K), LD4124.1 (K)
- new net COL25: LD1025.1 (K), LD1125.1 (K), LD1225.1 (K), LD1325.1 (K), LD1425.1 (K), LD1525.1 (K), LD1625.1 (K), LD1725.1 (K), LD1825.1 (K), LD1925.1 (K), LD2025.1 (K), LD2125.1 (K), LD2225.1 (K), LD2325.1 (K), LD2425.1 (K), LD2525.1 (K), LD2625.1 (K), LD2725.1 (K), LD2825.1 (K), LD2925.1 (K), LD3025.1 (K), LD3125.1 (K), LD3225.1 (K), LD3325.1 (K), LD3425.1 (K), LD3525.1 (K), LD3625.1 (K), LD3725.1 (K), LD3825.1 (K), LD3925.1 (K), LD4025.1 (K), LD4125.1 (K)
- new net COL26: LD1026.1 (K), LD1126.1 (K), LD1226.1 (K), LD1326.1 (K), LD1426.1 (K), LD1526.1 (K), LD1626.1 (K), LD1726.1 (K), LD1826.1 (K), LD1926.1 (K), LD2026.1 (K), LD2126.1 (K), LD2226.1 (K), LD2326.1 (K), LD2426.1 (K), LD2526.1 (K), LD2626.1 (K), LD2726.1 (K), LD2826.1 (K), LD2926.1 (K), LD3026.1 (K), LD3126.1 (K), LD3226.1 (K), LD3326.1 (K), LD3426.1 (K), LD3526.1 (K), LD3626.1 (K), LD3726.1 (K), LD3826.1 (K), LD3926.1 (K), LD4026.1 (K), LD4126.1 (K)
- new net COL27: LD1027.1 (K), LD1127.1 (K), LD1227.1 (K), LD1327.1 (K), LD1427.1 (K), LD1527.1 (K), LD1627.1 (K), LD1727.1 (K), LD1827.1 (K), LD1927.1 (K), LD2027.1 (K), LD2127.1 (K), LD2227.1 (K), LD2327.1 (K), LD2427.1 (K), LD2527.1 (K), LD2627.1 (K), LD2727.1 (K), LD2827.1 (K), LD2927.1 (K), LD3027.1 (K), LD3127.1 (K), LD3227.1 (K), LD3327.1 (K), LD3427.1 (K), LD3527.1 (K), LD3627.1 (K), LD3727.1 (K), LD3827.1 (K), LD3927.1 (K), LD4027.1 (K), LD4127.1 (K)
- new net COL28: LD1028.1 (K), LD1128.1 (K), LD1228.1 (K), LD1328.1 (K), LD1428.1 (K), LD1528.1 (K), LD1628.1 (K), LD1728.1 (K), LD1828.1 (K), LD1928.1 (K), LD2028.1 (K), LD2128.1 (K), LD2228.1 (K), LD2328.1 (K), LD2428.1 (K), LD2528.1 (K), LD2628.1 (K), LD2728.1 (K), LD2828.1 (K), LD2928.1 (K), LD3028.1 (K), LD3128.1 (K), LD3228.1 (K), LD3328.1 (K), LD3428.1 (K), LD3528.1 (K), LD3628.1 (K), LD3728.1 (K), LD3828.1 (K), LD3928.1 (K), LD4028.1 (K), LD4128.1 (K)
- new net COL29: LD1029.1 (K), LD1129.1 (K), LD1229.1 (K), LD1329.1 (K), LD1429.1 (K), LD1529.1 (K), LD1629.1 (K), LD1729.1 (K), LD1829.1 (K), LD1929.1 (K), LD2029.1 (K), LD2129.1 (K), LD2229.1 (K), LD2329.1 (K), LD2429.1 (K), LD2529.1 (K), LD2629.1 (K), LD2729.1 (K), LD2829.1 (K), LD2929.1 (K), LD3029.1 (K), LD3129.1 (K), LD3229.1 (K), LD3329.1 (K), LD3429.1 (K), LD3529.1 (K), LD3629.1 (K), LD3729.1 (K), LD3829.1 (K), LD3929.1 (K), LD4029.1 (K), LD4129.1 (K)
- new net COL3: LD1003.1 (K), LD1103.1 (K), LD1203.1 (K), LD1303.1 (K), LD1403.1 (K), LD1503.1 (K), LD1603.1 (K), LD1703.1 (K), LD1803.1 (K), LD1903.1 (K), LD2003.1 (K), LD2103.1 (K), LD2203.1 (K), LD2303.1 (K), LD2403.1 (K), LD2503.1 (K), LD2603.1 (K), LD2703.1 (K), LD2803.1 (K), LD2903.1 (K), LD3003.1 (K), LD3103.1 (K), LD3203.1 (K), LD3303.1 (K), LD3403.1 (K), LD3503.1 (K), LD3603.1 (K), LD3703.1 (K), LD3803.1 (K), LD3903.1 (K), LD4003.1 (K), LD4103.1 (K)
- new net COL30: LD1030.1 (K), LD1130.1 (K), LD1230.1 (K), LD1330.1 (K), LD1430.1 (K), LD1530.1 (K), LD1630.1 (K), LD1730.1 (K), LD1830.1 (K), LD1930.1 (K), LD2030.1 (K), LD2130.1 (K), LD2230.1 (K), LD2330.1 (K), LD2430.1 (K), LD2530.1 (K), LD2630.1 (K), LD2730.1 (K), LD2830.1 (K), LD2930.1 (K), LD3030.1 (K), LD3130.1 (K), LD3230.1 (K), LD3330.1 (K), LD3430.1 (K), LD3530.1 (K), LD3630.1 (K), LD3730.1 (K), LD3830.1 (K), LD3930.1 (K), LD4030.1 (K), LD4130.1 (K)
- new net COL31: LD1031.1 (K), LD1131.1 (K), LD1231.1 (K), LD1331.1 (K), LD1431.1 (K), LD1531.1 (K), LD1631.1 (K), LD1731.1 (K), LD1831.1 (K), LD1931.1 (K), LD2031.1 (K), LD2131.1 (K), LD2231.1 (K), LD2331.1 (K), LD2431.1 (K), LD2531.1 (K), LD2631.1 (K), LD2731.1 (K), LD2831.1 (K), LD2931.1 (K), LD3031.1 (K), LD3131.1 (K), LD3231.1 (K), LD3331.1 (K), LD3431.1 (K), LD3531.1 (K), LD3631.1 (K), LD3731.1 (K), LD3831.1 (K), LD3931.1 (K), LD4031.1 (K), LD4131.1 (K)
- new net COL4: LD1004.1 (K), LD1104.1 (K), LD1204.1 (K), LD1304.1 (K), LD1404.1 (K), LD1504.1 (K), LD1604.1 (K), LD1704.1 (K), LD1804.1 (K), LD1904.1 (K), LD2004.1 (K), LD2104.1 (K), LD2204.1 (K), LD2304.1 (K), LD2404.1 (K), LD2504.1 (K), LD2604.1 (K), LD2704.1 (K), LD2804.1 (K), LD2904.1 (K), LD3004.1 (K), LD3104.1 (K), LD3204.1 (K), LD3304.1 (K), LD3404.1 (K), LD3504.1 (K), LD3604.1 (K), LD3704.1 (K), LD3804.1 (K), LD3904.1 (K), LD4004.1 (K), LD4104.1 (K)
- new net COL5: LD1005.1 (K), LD1105.1 (K), LD1205.1 (K), LD1305.1 (K), LD1405.1 (K), LD1505.1 (K), LD1605.1 (K), LD1705.1 (K), LD1805.1 (K), LD1905.1 (K), LD2005.1 (K), LD2105.1 (K), LD2205.1 (K), LD2305.1 (K), LD2405.1 (K), LD2505.1 (K), LD2605.1 (K), LD2705.1 (K), LD2805.1 (K), LD2905.1 (K), LD3005.1 (K), LD3105.1 (K), LD3205.1 (K), LD3305.1 (K), LD3405.1 (K), LD3505.1 (K), LD3605.1 (K), LD3705.1 (K), LD3805.1 (K), LD3905.1 (K), LD4005.1 (K), LD4105.1 (K)
- new net COL6: LD1006.1 (K), LD1106.1 (K), LD1206.1 (K), LD1306.1 (K), LD1406.1 (K), LD1506.1 (K), LD1606.1 (K), LD1706.1 (K), LD1806.1 (K), LD1906.1 (K), LD2006.1 (K), LD2106.1 (K), LD2206.1 (K), LD2306.1 (K), LD2406.1 (K), LD2506.1 (K), LD2606.1 (K), LD2706.1 (K), LD2806.1 (K), LD2906.1 (K), LD3006.1 (K), LD3106.1 (K), LD3206.1 (K), LD3306.1 (K), LD3406.1 (K), LD3506.1 (K), LD3606.1 (K), LD3706.1 (K), LD3806.1 (K), LD3906.1 (K), LD4006.1 (K), LD4106.1 (K)
- new net COL7: LD1007.1 (K), LD1107.1 (K), LD1207.1 (K), LD1307.1 (K), LD1407.1 (K), LD1507.1 (K), LD1607.1 (K), LD1707.1 (K), LD1807.1 (K), LD1907.1 (K), LD2007.1 (K), LD2107.1 (K), LD2207.1 (K), LD2307.1 (K), LD2407.1 (K), LD2507.1 (K), LD2607.1 (K), LD2707.1 (K), LD2807.1 (K), LD2907.1 (K), LD3007.1 (K), LD3107.1 (K), LD3207.1 (K), LD3307.1 (K), LD3407.1 (K), LD3507.1 (K), LD3607.1 (K), LD3707.1 (K), LD3807.1 (K), LD3907.1 (K), LD4007.1 (K), LD4107.1 (K)
- new net COL8: LD1008.1 (K), LD1108.1 (K), LD1208.1 (K), LD1308.1 (K), LD1408.1 (K), LD1508.1 (K), LD1608.1 (K), LD1708.1 (K), LD1808.1 (K), LD1908.1 (K), LD2008.1 (K), LD2108.1 (K), LD2208.1 (K), LD2308.1 (K), LD2408.1 (K), LD2508.1 (K), LD2608.1 (K), LD2708.1 (K), LD2808.1 (K), LD2908.1 (K), LD3008.1 (K), LD3108.1 (K), LD3208.1 (K), LD3308.1 (K), LD3408.1 (K), LD3508.1 (K), LD3608.1 (K), LD3708.1 (K), LD3808.1 (K), LD3908.1 (K), LD4008.1 (K), LD4108.1 (K)
- new net COL9: LD1009.1 (K), LD1109.1 (K), LD1209.1 (K), LD1309.1 (K), LD1409.1 (K), LD1509.1 (K), LD1609.1 (K), LD1709.1 (K), LD1809.1 (K), LD1909.1 (K), LD2009.1 (K), LD2109.1 (K), LD2209.1 (K), LD2309.1 (K), LD2409.1 (K), LD2509.1 (K), LD2609.1 (K), LD2709.1 (K), LD2809.1 (K), LD2909.1 (K), LD3009.1 (K), LD3109.1 (K), LD3209.1 (K), LD3309.1 (K), LD3409.1 (K), LD3509.1 (K), LD3609.1 (K), LD3709.1 (K), LD3809.1 (K), LD3909.1 (K), LD4009.1 (K), LD4109.1 (K)
- new net ROW0: LD1000.2 (A), LD1001.2 (A), LD1002.2 (A), LD1003.2 (A), LD1004.2 (A), LD1005.2 (A), LD1006.2 (A), LD1007.2 (A), LD1008.2 (A), LD1009.2 (A), LD1010.2 (A), LD1011.2 (A), LD1012.2 (A), LD1013.2 (A), LD1014.2 (A), LD1015.2 (A), LD1016.2 (A), LD1017.2 (A), LD1018.2 (A), LD1019.2 (A), LD1020.2 (A), LD1021.2 (A), LD1022.2 (A), LD1023.2 (A), LD1024.2 (A), LD1025.2 (A), LD1026.2 (A), LD1027.2 (A), LD1028.2 (A), LD1029.2 (A), LD1030.2 (A), LD1031.2 (A)
- new net ROW1: LD1100.2 (A), LD1101.2 (A), LD1102.2 (A), LD1103.2 (A), LD1104.2 (A), LD1105.2 (A), LD1106.2 (A), LD1107.2 (A), LD1108.2 (A), LD1109.2 (A), LD1110.2 (A), LD1111.2 (A), LD1112.2 (A), LD1113.2 (A), LD1114.2 (A), LD1115.2 (A), LD1116.2 (A), LD1117.2 (A), LD1118.2 (A), LD1119.2 (A), LD1120.2 (A), LD1121.2 (A), LD1122.2 (A), LD1123.2 (A), LD1124.2 (A), LD1125.2 (A), LD1126.2 (A), LD1127.2 (A), LD1128.2 (A), LD1129.2 (A), LD1130.2 (A), LD1131.2 (A)
- new net ROW10: LD2000.2 (A), LD2001.2 (A), LD2002.2 (A), LD2003.2 (A), LD2004.2 (A), LD2005.2 (A), LD2006.2 (A), LD2007.2 (A), LD2008.2 (A), LD2009.2 (A), LD2010.2 (A), LD2011.2 (A), LD2012.2 (A), LD2013.2 (A), LD2014.2 (A), LD2015.2 (A), LD2016.2 (A), LD2017.2 (A), LD2018.2 (A), LD2019.2 (A), LD2020.2 (A), LD2021.2 (A), LD2022.2 (A), LD2023.2 (A), LD2024.2 (A), LD2025.2 (A), LD2026.2 (A), LD2027.2 (A), LD2028.2 (A), LD2029.2 (A), LD2030.2 (A), LD2031.2 (A)
- new net ROW11: LD2100.2 (A), LD2101.2 (A), LD2102.2 (A), LD2103.2 (A), LD2104.2 (A), LD2105.2 (A), LD2106.2 (A), LD2107.2 (A), LD2108.2 (A), LD2109.2 (A), LD2110.2 (A), LD2111.2 (A), LD2112.2 (A), LD2113.2 (A), LD2114.2 (A), LD2115.2 (A), LD2116.2 (A), LD2117.2 (A), LD2118.2 (A), LD2119.2 (A), LD2120.2 (A), LD2121.2 (A), LD2122.2 (A), LD2123.2 (A), LD2124.2 (A), LD2125.2 (A), LD2126.2 (A), LD2127.2 (A), LD2128.2 (A), LD2129.2 (A), LD2130.2 (A), LD2131.2 (A)
- new net ROW12: LD2200.2 (A), LD2201.2 (A), LD2202.2 (A), LD2203.2 (A), LD2204.2 (A), LD2205.2 (A), LD2206.2 (A), LD2207.2 (A), LD2208.2 (A), LD2209.2 (A), LD2210.2 (A), LD2211.2 (A), LD2212.2 (A), LD2213.2 (A), LD2214.2 (A), LD2215.2 (A), LD2216.2 (A), LD2217.2 (A), LD2218.2 (A), LD2219.2 (A), LD2220.2 (A), LD2221.2 (A), LD2222.2 (A), LD2223.2 (A), LD2224.2 (A), LD2225.2 (A), LD2226.2 (A), LD2227.2 (A), LD2228.2 (A), LD2229.2 (A), LD2230.2 (A), LD2231.2 (A)
- new net ROW13: LD2300.2 (A), LD2301.2 (A), LD2302.2 (A), LD2303.2 (A), LD2304.2 (A), LD2305.2 (A), LD2306.2 (A), LD2307.2 (A), LD2308.2 (A), LD2309.2 (A), LD2310.2 (A), LD2311.2 (A), LD2312.2 (A), LD2313.2 (A), LD2314.2 (A), LD2315.2 (A), LD2316.2 (A), LD2317.2 (A), LD2318.2 (A), LD2319.2 (A), LD2320.2 (A), LD2321.2 (A), LD2322.2 (A), LD2323.2 (A), LD2324.2 (A), LD2325.2 (A), LD2326.2 (A), LD2327.2 (A), LD2328.2 (A), LD2329.2 (A), LD2330.2 (A), LD2331.2 (A)
- new net ROW14: LD2400.2 (A), LD2401.2 (A), LD2402.2 (A), LD2403.2 (A), LD2404.2 (A), LD2405.2 (A), LD2406.2 (A), LD2407.2 (A), LD2408.2 (A), LD2409.2 (A), LD2410.2 (A), LD2411.2 (A), LD2412.2 (A), LD2413.2 (A), LD2414.2 (A), LD2415.2 (A), LD2416.2 (A), LD2417.2 (A), LD2418.2 (A), LD2419.2 (A), LD2420.2 (A), LD2421.2 (A), LD2422.2 (A), LD2423.2 (A), LD2424.2 (A), LD2425.2 (A), LD2426.2 (A), LD2427.2 (A), LD2428.2 (A), LD2429.2 (A), LD2430.2 (A), LD2431.2 (A)
- new net ROW15: LD2500.2 (A), LD2501.2 (A), LD2502.2 (A), LD2503.2 (A), LD2504.2 (A), LD2505.2 (A), LD2506.2 (A), LD2507.2 (A), LD2508.2 (A), LD2509.2 (A), LD2510.2 (A), LD2511.2 (A), LD2512.2 (A), LD2513.2 (A), LD2514.2 (A), LD2515.2 (A), LD2516.2 (A), LD2517.2 (A), LD2518.2 (A), LD2519.2 (A), LD2520.2 (A), LD2521.2 (A), LD2522.2 (A), LD2523.2 (A), LD2524.2 (A), LD2525.2 (A), LD2526.2 (A), LD2527.2 (A), LD2528.2 (A), LD2529.2 (A), LD2530.2 (A), LD2531.2 (A)
- new net ROW16: LD2600.2 (A), LD2601.2 (A), LD2602.2 (A), LD2603.2 (A), LD2604.2 (A), LD2605.2 (A), LD2606.2 (A), LD2607.2 (A), LD2608.2 (A), LD2609.2 (A), LD2610.2 (A), LD2611.2 (A), LD2612.2 (A), LD2613.2 (A), LD2614.2 (A), LD2615.2 (A), LD2616.2 (A), LD2617.2 (A), LD2618.2 (A), LD2619.2 (A), LD2620.2 (A), LD2621.2 (A), LD2622.2 (A), LD2623.2 (A), LD2624.2 (A), LD2625.2 (A), LD2626.2 (A), LD2627.2 (A), LD2628.2 (A), LD2629.2 (A), LD2630.2 (A), LD2631.2 (A)
- new net ROW17: LD2700.2 (A), LD2701.2 (A), LD2702.2 (A), LD2703.2 (A), LD2704.2 (A), LD2705.2 (A), LD2706.2 (A), LD2707.2 (A), LD2708.2 (A), LD2709.2 (A), LD2710.2 (A), LD2711.2 (A), LD2712.2 (A), LD2713.2 (A), LD2714.2 (A), LD2715.2 (A), LD2716.2 (A), LD2717.2 (A), LD2718.2 (A), LD2719.2 (A), LD2720.2 (A), LD2721.2 (A), LD2722.2 (A), LD2723.2 (A), LD2724.2 (A), LD2725.2 (A), LD2726.2 (A), LD2727.2 (A), LD2728.2 (A), LD2729.2 (A), LD2730.2 (A), LD2731.2 (A)
- new net ROW18: LD2800.2 (A), LD2801.2 (A), LD2802.2 (A), LD2803.2 (A), LD2804.2 (A), LD2805.2 (A), LD2806.2 (A), LD2807.2 (A), LD2808.2 (A), LD2809.2 (A), LD2810.2 (A), LD2811.2 (A), LD2812.2 (A), LD2813.2 (A), LD2814.2 (A), LD2815.2 (A), LD2816.2 (A), LD2817.2 (A), LD2818.2 (A), LD2819.2 (A), LD2820.2 (A), LD2821.2 (A), LD2822.2 (A), LD2823.2 (A), LD2824.2 (A), LD2825.2 (A), LD2826.2 (A), LD2827.2 (A), LD2828.2 (A), LD2829.2 (A), LD2830.2 (A), LD2831.2 (A)
- new net ROW19: LD2900.2 (A), LD2901.2 (A), LD2902.2 (A), LD2903.2 (A), LD2904.2 (A), LD2905.2 (A), LD2906.2 (A), LD2907.2 (A), LD2908.2 (A), LD2909.2 (A), LD2910.2 (A), LD2911.2 (A), LD2912.2 (A), LD2913.2 (A), LD2914.2 (A), LD2915.2 (A), LD2916.2 (A), LD2917.2 (A), LD2918.2 (A), LD2919.2 (A), LD2920.2 (A), LD2921.2 (A), LD2922.2 (A), LD2923.2 (A), LD2924.2 (A), LD2925.2 (A), LD2926.2 (A), LD2927.2 (A), LD2928.2 (A), LD2929.2 (A), LD2930.2 (A), LD2931.2 (A)
- new net ROW2: LD1200.2 (A), LD1201.2 (A), LD1202.2 (A), LD1203.2 (A), LD1204.2 (A), LD1205.2 (A), LD1206.2 (A), LD1207.2 (A), LD1208.2 (A), LD1209.2 (A), LD1210.2 (A), LD1211.2 (A), LD1212.2 (A), LD1213.2 (A), LD1214.2 (A), LD1215.2 (A), LD1216.2 (A), LD1217.2 (A), LD1218.2 (A), LD1219.2 (A), LD1220.2 (A), LD1221.2 (A), LD1222.2 (A), LD1223.2 (A), LD1224.2 (A), LD1225.2 (A), LD1226.2 (A), LD1227.2 (A), LD1228.2 (A), LD1229.2 (A), LD1230.2 (A), LD1231.2 (A)
- new net ROW20: LD3000.2 (A), LD3001.2 (A), LD3002.2 (A), LD3003.2 (A), LD3004.2 (A), LD3005.2 (A), LD3006.2 (A), LD3007.2 (A), LD3008.2 (A), LD3009.2 (A), LD3010.2 (A), LD3011.2 (A), LD3012.2 (A), LD3013.2 (A), LD3014.2 (A), LD3015.2 (A), LD3016.2 (A), LD3017.2 (A), LD3018.2 (A), LD3019.2 (A), LD3020.2 (A), LD3021.2 (A), LD3022.2 (A), LD3023.2 (A), LD3024.2 (A), LD3025.2 (A), LD3026.2 (A), LD3027.2 (A), LD3028.2 (A), LD3029.2 (A), LD3030.2 (A), LD3031.2 (A)
- new net ROW21: LD3100.2 (A), LD3101.2 (A), LD3102.2 (A), LD3103.2 (A), LD3104.2 (A), LD3105.2 (A), LD3106.2 (A), LD3107.2 (A), LD3108.2 (A), LD3109.2 (A), LD3110.2 (A), LD3111.2 (A), LD3112.2 (A), LD3113.2 (A), LD3114.2 (A), LD3115.2 (A), LD3116.2 (A), LD3117.2 (A), LD3118.2 (A), LD3119.2 (A), LD3120.2 (A), LD3121.2 (A), LD3122.2 (A), LD3123.2 (A), LD3124.2 (A), LD3125.2 (A), LD3126.2 (A), LD3127.2 (A), LD3128.2 (A), LD3129.2 (A), LD3130.2 (A), LD3131.2 (A)
- new net ROW22: LD3200.2 (A), LD3201.2 (A), LD3202.2 (A), LD3203.2 (A), LD3204.2 (A), LD3205.2 (A), LD3206.2 (A), LD3207.2 (A), LD3208.2 (A), LD3209.2 (A), LD3210.2 (A), LD3211.2 (A), LD3212.2 (A), LD3213.2 (A), LD3214.2 (A), LD3215.2 (A), LD3216.2 (A), LD3217.2 (A), LD3218.2 (A), LD3219.2 (A), LD3220.2 (A), LD3221.2 (A), LD3222.2 (A), LD3223.2 (A), LD3224.2 (A), LD3225.2 (A), LD3226.2 (A), LD3227.2 (A), LD3228.2 (A), LD3229.2 (A), LD3230.2 (A), LD3231.2 (A)
- new net ROW23: LD3300.2 (A), LD3301.2 (A), LD3302.2 (A), LD3303.2 (A), LD3304.2 (A), LD3305.2 (A), LD3306.2 (A), LD3307.2 (A), LD3308.2 (A), LD3309.2 (A), LD3310.2 (A), LD3311.2 (A), LD3312.2 (A), LD3313.2 (A), LD3314.2 (A), LD3315.2 (A), LD3316.2 (A), LD3317.2 (A), LD3318.2 (A), LD3319.2 (A), LD3320.2 (A), LD3321.2 (A), LD3322.2 (A), LD3323.2 (A), LD3324.2 (A), LD3325.2 (A), LD3326.2 (A), LD3327.2 (A), LD3328.2 (A), LD3329.2 (A), LD3330.2 (A), LD3331.2 (A)
- new net ROW24: LD3400.2 (A), LD3401.2 (A), LD3402.2 (A), LD3403.2 (A), LD3404.2 (A), LD3405.2 (A), LD3406.2 (A), LD3407.2 (A), LD3408.2 (A), LD3409.2 (A), LD3410.2 (A), LD3411.2 (A), LD3412.2 (A), LD3413.2 (A), LD3414.2 (A), LD3415.2 (A), LD3416.2 (A), LD3417.2 (A), LD3418.2 (A), LD3419.2 (A), LD3420.2 (A), LD3421.2 (A), LD3422.2 (A), LD3423.2 (A), LD3424.2 (A), LD3425.2 (A), LD3426.2 (A), LD3427.2 (A), LD3428.2 (A), LD3429.2 (A), LD3430.2 (A), LD3431.2 (A)
- new net ROW25: LD3500.2 (A), LD3501.2 (A), LD3502.2 (A), LD3503.2 (A), LD3504.2 (A), LD3505.2 (A), LD3506.2 (A), LD3507.2 (A), LD3508.2 (A), LD3509.2 (A), LD3510.2 (A), LD3511.2 (A), LD3512.2 (A), LD3513.2 (A), LD3514.2 (A), LD3515.2 (A), LD3516.2 (A), LD3517.2 (A), LD3518.2 (A), LD3519.2 (A), LD3520.2 (A), LD3521.2 (A), LD3522.2 (A), LD3523.2 (A), LD3524.2 (A), LD3525.2 (A), LD3526.2 (A), LD3527.2 (A), LD3528.2 (A), LD3529.2 (A), LD3530.2 (A), LD3531.2 (A)
- new net ROW26: LD3600.2 (A), LD3601.2 (A), LD3602.2 (A), LD3603.2 (A), LD3604.2 (A), LD3605.2 (A), LD3606.2 (A), LD3607.2 (A), LD3608.2 (A), LD3609.2 (A), LD3610.2 (A), LD3611.2 (A), LD3612.2 (A), LD3613.2 (A), LD3614.2 (A), LD3615.2 (A), LD3616.2 (A), LD3617.2 (A), LD3618.2 (A), LD3619.2 (A), LD3620.2 (A), LD3621.2 (A), LD3622.2 (A), LD3623.2 (A), LD3624.2 (A), LD3625.2 (A), LD3626.2 (A), LD3627.2 (A), LD3628.2 (A), LD3629.2 (A), LD3630.2 (A), LD3631.2 (A)
- new net ROW27: LD3700.2 (A), LD3701.2 (A), LD3702.2 (A), LD3703.2 (A), LD3704.2 (A), LD3705.2 (A), LD3706.2 (A), LD3707.2 (A), LD3708.2 (A), LD3709.2 (A), LD3710.2 (A), LD3711.2 (A), LD3712.2 (A), LD3713.2 (A), LD3714.2 (A), LD3715.2 (A), LD3716.2 (A), LD3717.2 (A), LD3718.2 (A), LD3719.2 (A), LD3720.2 (A), LD3721.2 (A), LD3722.2 (A), LD3723.2 (A), LD3724.2 (A), LD3725.2 (A), LD3726.2 (A), LD3727.2 (A), LD3728.2 (A), LD3729.2 (A), LD3730.2 (A), LD3731.2 (A)
- new net ROW28: LD3800.2 (A), LD3801.2 (A), LD3802.2 (A), LD3803.2 (A), LD3804.2 (A), LD3805.2 (A), LD3806.2 (A), LD3807.2 (A), LD3808.2 (A), LD3809.2 (A), LD3810.2 (A), LD3811.2 (A), LD3812.2 (A), LD3813.2 (A), LD3814.2 (A), LD3815.2 (A), LD3816.2 (A), LD3817.2 (A), LD3818.2 (A), LD3819.2 (A), LD3820.2 (A), LD3821.2 (A), LD3822.2 (A), LD3823.2 (A), LD3824.2 (A), LD3825.2 (A), LD3826.2 (A), LD3827.2 (A), LD3828.2 (A), LD3829.2 (A), LD3830.2 (A), LD3831.2 (A)
- new net ROW29: LD3900.2 (A), LD3901.2 (A), LD3902.2 (A), LD3903.2 (A), LD3904.2 (A), LD3905.2 (A), LD3906.2 (A), LD3907.2 (A), LD3908.2 (A), LD3909.2 (A), LD3910.2 (A), LD3911.2 (A), LD3912.2 (A), LD3913.2 (A), LD3914.2 (A), LD3915.2 (A), LD3916.2 (A), LD3917.2 (A), LD3918.2 (A), LD3919.2 (A), LD3920.2 (A), LD3921.2 (A), LD3922.2 (A), LD3923.2 (A), LD3924.2 (A), LD3925.2 (A), LD3926.2 (A), LD3927.2 (A), LD3928.2 (A), LD3929.2 (A), LD3930.2 (A), LD3931.2 (A)
- new net ROW3: LD1300.2 (A), LD1301.2 (A), LD1302.2 (A), LD1303.2 (A), LD1304.2 (A), LD1305.2 (A), LD1306.2 (A), LD1307.2 (A), LD1308.2 (A), LD1309.2 (A), LD1310.2 (A), LD1311.2 (A), LD1312.2 (A), LD1313.2 (A), LD1314.2 (A), LD1315.2 (A), LD1316.2 (A), LD1317.2 (A), LD1318.2 (A), LD1319.2 (A), LD1320.2 (A), LD1321.2 (A), LD1322.2 (A), LD1323.2 (A), LD1324.2 (A), LD1325.2 (A), LD1326.2 (A), LD1327.2 (A), LD1328.2 (A), LD1329.2 (A), LD1330.2 (A), LD1331.2 (A)
- new net ROW30: LD4000.2 (A), LD4001.2 (A), LD4002.2 (A), LD4003.2 (A), LD4004.2 (A), LD4005.2 (A), LD4006.2 (A), LD4007.2 (A), LD4008.2 (A), LD4009.2 (A), LD4010.2 (A), LD4011.2 (A), LD4012.2 (A), LD4013.2 (A), LD4014.2 (A), LD4015.2 (A), LD4016.2 (A), LD4017.2 (A), LD4018.2 (A), LD4019.2 (A), LD4020.2 (A), LD4021.2 (A), LD4022.2 (A), LD4023.2 (A), LD4024.2 (A), LD4025.2 (A), LD4026.2 (A), LD4027.2 (A), LD4028.2 (A), LD4029.2 (A), LD4030.2 (A), LD4031.2 (A)
- new net ROW31: LD4100.2 (A), LD4101.2 (A), LD4102.2 (A), LD4103.2 (A), LD4104.2 (A), LD4105.2 (A), LD4106.2 (A), LD4107.2 (A), LD4108.2 (A), LD4109.2 (A), LD4110.2 (A), LD4111.2 (A), LD4112.2 (A), LD4113.2 (A), LD4114.2 (A), LD4115.2 (A), LD4116.2 (A), LD4117.2 (A), LD4118.2 (A), LD4119.2 (A), LD4120.2 (A), LD4121.2 (A), LD4122.2 (A), LD4123.2 (A), LD4124.2 (A), LD4125.2 (A), LD4126.2 (A), LD4127.2 (A), LD4128.2 (A), LD4129.2 (A), LD4130.2 (A), LD4131.2 (A)
- new net ROW4: LD1400.2 (A), LD1401.2 (A), LD1402.2 (A), LD1403.2 (A), LD1404.2 (A), LD1405.2 (A), LD1406.2 (A), LD1407.2 (A), LD1408.2 (A), LD1409.2 (A), LD1410.2 (A), LD1411.2 (A), LD1412.2 (A), LD1413.2 (A), LD1414.2 (A), LD1415.2 (A), LD1416.2 (A), LD1417.2 (A), LD1418.2 (A), LD1419.2 (A), LD1420.2 (A), LD1421.2 (A), LD1422.2 (A), LD1423.2 (A), LD1424.2 (A), LD1425.2 (A), LD1426.2 (A), LD1427.2 (A), LD1428.2 (A), LD1429.2 (A), LD1430.2 (A), LD1431.2 (A)
- new net ROW5: LD1500.2 (A), LD1501.2 (A), LD1502.2 (A), LD1503.2 (A), LD1504.2 (A), LD1505.2 (A), LD1506.2 (A), LD1507.2 (A), LD1508.2 (A), LD1509.2 (A), LD1510.2 (A), LD1511.2 (A), LD1512.2 (A), LD1513.2 (A), LD1514.2 (A), LD1515.2 (A), LD1516.2 (A), LD1517.2 (A), LD1518.2 (A), LD1519.2 (A), LD1520.2 (A), LD1521.2 (A), LD1522.2 (A), LD1523.2 (A), LD1524.2 (A), LD1525.2 (A), LD1526.2 (A), LD1527.2 (A), LD1528.2 (A), LD1529.2 (A), LD1530.2 (A), LD1531.2 (A)
- new net ROW6: LD1600.2 (A), LD1601.2 (A), LD1602.2 (A), LD1603.2 (A), LD1604.2 (A), LD1605.2 (A), LD1606.2 (A), LD1607.2 (A), LD1608.2 (A), LD1609.2 (A), LD1610.2 (A), LD1611.2 (A), LD1612.2 (A), LD1613.2 (A), LD1614.2 (A), LD1615.2 (A), LD1616.2 (A), LD1617.2 (A), LD1618.2 (A), LD1619.2 (A), LD1620.2 (A), LD1621.2 (A), LD1622.2 (A), LD1623.2 (A), LD1624.2 (A), LD1625.2 (A), LD1626.2 (A), LD1627.2 (A), LD1628.2 (A), LD1629.2 (A), LD1630.2 (A), LD1631.2 (A)
- new net ROW7: LD1700.2 (A), LD1701.2 (A), LD1702.2 (A), LD1703.2 (A), LD1704.2 (A), LD1705.2 (A), LD1706.2 (A), LD1707.2 (A), LD1708.2 (A), LD1709.2 (A), LD1710.2 (A), LD1711.2 (A), LD1712.2 (A), LD1713.2 (A), LD1714.2 (A), LD1715.2 (A), LD1716.2 (A), LD1717.2 (A), LD1718.2 (A), LD1719.2 (A), LD1720.2 (A), LD1721.2 (A), LD1722.2 (A), LD1723.2 (A), LD1724.2 (A), LD1725.2 (A), LD1726.2 (A), LD1727.2 (A), LD1728.2 (A), LD1729.2 (A), LD1730.2 (A), LD1731.2 (A)
- new net ROW8: LD1800.2 (A), LD1801.2 (A), LD1802.2 (A), LD1803.2 (A), LD1804.2 (A), LD1805.2 (A), LD1806.2 (A), LD1807.2 (A), LD1808.2 (A), LD1809.2 (A), LD1810.2 (A), LD1811.2 (A), LD1812.2 (A), LD1813.2 (A), LD1814.2 (A), LD1815.2 (A), LD1816.2 (A), LD1817.2 (A), LD1818.2 (A), LD1819.2 (A), LD1820.2 (A), LD1821.2 (A), LD1822.2 (A), LD1823.2 (A), LD1824.2 (A), LD1825.2 (A), LD1826.2 (A), LD1827.2 (A), LD1828.2 (A), LD1829.2 (A), LD1830.2 (A), LD1831.2 (A)
- new net ROW9: LD1900.2 (A), LD1901.2 (A), LD1902.2 (A), LD1903.2 (A), LD1904.2 (A), LD1905.2 (A), LD1906.2 (A), LD1907.2 (A), LD1908.2 (A), LD1909.2 (A), LD1910.2 (A), LD1911.2 (A), LD1912.2 (A), LD1913.2 (A), LD1914.2 (A), LD1915.2 (A), LD1916.2 (A), LD1917.2 (A), LD1918.2 (A), LD1919.2 (A), LD1920.2 (A), LD1921.2 (A), LD1922.2 (A), LD1923.2 (A), LD1924.2 (A), LD1925.2 (A), LD1926.2 (A), LD1927.2 (A), LD1928.2 (A), LD1929.2 (A), LD1930.2 (A), LD1931.2 (A)
Other:
- note added: "LED matrix (Rev A) - design notes 32 x 32 = 1024 LEDs, common-anode rows: LD(1000 + 100 x row + column), anode to ROWn (high-side AO3401A), cathode to COLn (TLC59283 sink). One row on at a time (1:32). LED part, pitch and peak current are PROTOTYPE-DEPENDENT (OD-03, QR screening); KT-0603W 0603 at 2.0 mm pitch is the current candidate. Front side of the board, with the two buttons when they fit (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"

Commit message: hw: start the Rev A layout with placement and matrix routing (#13)
* docs: record Raytac's USB decoupling reply and VBUS limit

Raytac R&D confirmed in writing that the DECUSB capacitor for the USB
regulator is inside the MDBT53 modules, and that the 4.7 µF behind 2.2 Ω
in their reference circuit is C_VBUS (C402/R401 on this board).

The attach-inrush fallback now stays within the nRF5340 limit of 6 Ω DC
VBUS source resistance, including the cable, when VDDH is not supplied
from VBUS: R401 stays at or below 4.7 Ω, and a smaller C402 is checked
against the nRF5340 VBUS decoupling requirement before it is fitted.

* hw: add layout footprints for LEDs, NFC coil, test pads and mic

The matrix LED footprint follows KENTO's suggested 0603 pad (0.70 x
0.70 mm, 0.70 mm gap). Pad 1 is the cathode, marked by a chamfered pad,
and the courtyard keeps its true size.

The NFC coil is the computed 30 x 25 mm, 6-turn coil (0.4 mm track,
0.3 mm gap) on F.Cu with an In1.Cu crossover. Its corners are chamfered
so the outer turn clears the 3 mm board corner, and a net tie joins its
two pads.

Adds a 0.8 mm test pad. The microphone's acoustic hole goes from 0.8 to
0.6 mm, still within Knowles' 0.6-1.0 mm, so the ground ring keeps the
fabricator's 0.2 mm clearance to an unplated hole.

* hw: add 3D models for all assembled parts

Uses KiCad library models where the pads and body match: SOT-563,
Coilcraft XAL4020, Murata DFE201610P scaled to 1.2 mm, TS-1088 and
Knowles SPH0645.

The TI DLA0010A and RYK0018A, NXP SOT902-3, MDBT53-P1M and HRO USB-C
get envelope STEP models built from the fab outline and the datasheet
maximum height. They are meant for clearance and carrier checks only.

The HRO footprint is copied into the project library because KiCad
ships no model for it.

* hw: apply layout footprint and test-point changes to the schematic

The matrix LEDs use the KENTO-pattern footprint, L1101 the PCB coil,
MK1001 the 0.6 mm hole footprint and J301 the project HRO copy.

Removes test p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
Parts:
- LD1000, LD1001, LD1002, LD1003, LD1004, LD1005, LD1006, LD1007, LD1008, LD1009, LD1010, LD1011, LD1012, LD1013, LD1014, LD1015, LD1016, LD1017, LD1018, LD1019, LD1020, LD1021, LD1022, LD1023, LD1024, LD1025, LD1026, LD1027, LD1028, LD1029, LD1030, LD1031, LD1100, LD1101, LD1102, LD1103, LD1104, LD1105, LD1106, LD1107, LD1108, LD1109, LD1110, LD1111, LD1112, LD1113, LD1114, LD1115, LD1116, LD1117, LD1118, LD1119, LD1120, LD1121, LD1122, LD1123, LD1124, LD1125, LD1126, LD1127, LD1128, LD1129, LD1130, LD1131, LD1200, LD1201, LD1202, LD1203, LD1204, LD1205, LD1206, LD1207, LD1208, LD1209, LD1210, LD1211, LD1212, LD1213, LD1214, LD1215, LD1216, LD1217, LD1218, LD1219, LD1220, LD1221, LD1222, LD1223, LD1224, LD1225, LD1226, LD1227, LD1228, LD1229, LD1230, LD1231, LD1300, LD1301, LD1302, LD1303, LD1304, LD1305, LD1306, LD1307, LD1308, LD1309, LD1310, LD1311, LD1312, LD1313, LD1314, LD1315, LD1316, LD1317, LD1318, LD1319, LD1320, LD1321, LD1322, LD1323, LD1324, LD1325, LD1326, LD1327, LD1328, LD1329, LD1330, LD1331, LD1400, LD1401, LD1402, LD1403, LD1404, LD1405, LD1406, LD1407, LD1408, LD1409, LD1410, LD1411, LD1412, LD1413, LD1414, LD1415, LD1416, LD1417, LD1418, LD1419, LD1420, LD1421, LD1422, LD1423, LD1424, LD1425, LD1426, LD1427, LD1428, LD1429, LD1430, LD1431, LD1500, LD1501, LD1502, LD1503, LD1504, LD1505, LD1506, LD1507, LD1508, LD1509, LD1510, LD1511, LD1512, LD1513, LD1514, LD1515, LD1516, LD1517, LD1518, LD1519, LD1520, LD1521, LD1522, LD1523, LD1524, LD1525, LD1526, LD1527, LD1528, LD1529, LD1530, LD1531, LD1600, LD1601, LD1602, LD1603, LD1604, LD1605, LD1606, LD1607, LD1608, LD1609, LD1610, LD1611, LD1612, LD1613, LD1614, LD1615, LD1616, LD1617, LD1618, LD1619, LD1620, LD1621, LD1622, LD1623, LD1624, LD1625, LD1626, LD1627, LD1628, LD1629, LD1630, LD1631, LD1700, LD1701, LD1702, LD1703, LD1704, LD1705, LD1706, LD1707, LD1708, LD1709, LD1710, LD1711, LD1712, LD1713, LD1714, LD1715, LD1716, LD1717, LD1718, LD1719, LD1720, LD1721, LD1722, LD1723, LD1724, LD1725, LD1726, LD1727, LD1728, LD1729, LD1730, LD1731, LD1800, LD1801, LD1802, LD1803, LD1804, LD1805, LD1806, LD1807, LD1808, LD1809, LD1810, LD1811, LD1812, LD1813, LD1814, LD1815, LD1816, LD1817, LD1818, LD1819, LD1820, LD1821, LD1822, LD1823, LD1824, LD1825, LD1826, LD1827, LD1828, LD1829, LD1830, LD1831, LD1900, LD1901, LD1902, LD1903, LD1904, LD1905, LD1906, LD1907, LD1908, LD1909, LD1910, LD1911, LD1912, LD1913, LD1914, LD1915, LD1916, LD1917, LD1918, LD1919, LD1920, LD1921, LD1922, LD1923, LD1924, LD1925, LD1926, LD1927, LD1928, LD1929, LD1930, LD1931, LD2000, LD2001, LD2002, LD2003, LD2004, LD2005, LD2006, LD2007, LD2008, LD2009, LD2010, LD2011, LD2012, LD2013, LD2014, LD2015, LD2016, LD2017, LD2018, LD2019, LD2020, LD2021, LD2022, LD2023, LD2024, LD2025, LD2026, LD2027, LD2028, LD2029, LD2030, LD2031, LD2100, LD2101, LD2102, LD2103, LD2104, LD2105, LD2106, LD2107, LD2108, LD2109, LD2110, LD2111, LD2112, LD2113, LD2114, LD2115, LD2116, LD2117, LD2118, LD2119, LD2120, LD2121, LD2122, LD2123, LD2124, LD2125, LD2126, LD2127, LD2128, LD2129, LD2130, LD2131, LD2200, LD2201, LD2202, LD2203, LD2204, LD2205, LD2206, LD2207, LD2208, LD2209, LD2210, LD2211, LD2212, LD2213, LD2214, LD2215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: footprint LED_SMD:LED_0603_1608Metric -> smart-led-badge:LED_0603_KENTO_KT-0603; Note Matrix LED PROTOTYPE-DEPENDENT (OD-03); front side, 2.0 mm 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 -> Matrix LED, selected on the KENTO datasheet (2026-10-08); f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
