File: hardware/sheets/imu.kicad_sch (KiCad schematic)
At the start: 0 parts

Commit message: hw: draw UI, IMU, microphone and NFC sheets
IMU: ICM-42688-P on the shared I2C1 bus at 0x68, bypassed as TDK's
application circuit specifies, reserved pins to ground, and unfitted
links for the SPI fallback.

Microphone: SPH0641LM4H-1 with a C0G bypass capacitor (Knowles advises
against class 2 dielectrics next to the part), a 0 ohm supply link for
current measurement, series options on clock and data, and SELECT to
ground.

NFC: NT3H2111W0FHKH powered from the NFC_PWR GPIO with its bus and
field-detect pull-ups, the PCB coil as a non-BOM part, two unfitted
tuning capacitor positions and test points for bus timing.

UI: two tact switches to ground with unfitted external pull-ups and a
red status LED.

The labels these sheets connect no longer need ERC exclusions. NFC_PWR
gets a reviewed exclusion: a GPIO drives the tag supply by design.
Parts:
- added C901: 100nF, Capacitor_SMD:C_0402_1005Metric, symbol Device:C
- added C902: 2.2uF X7R, Capacitor_SMD:C_0603_1608Metric, symbol Device:C
- added C903: 10nF, Capacitor_SMD:C_0402_1005Metric, symbol Device:C
- added R901, R902: 10k, Resistor_SMD:R_0402_1005Metric, symbol Device:R
- added R903, R904: DNP, Resistor_SMD:R_0402_1005Metric, symbol Device:R
- added U901: ICM-42688-P, Package_LGA:LGA-14_3x2.5mm_P0.5mm_LayoutBorder3x4y, symbol smart-led-badge:ICM-42688-P
Connections:
- new net +3V3: C901.1, C902.1, C903.1, R901.2, U901.5 (VDDIO), U901.8 (VDD)
- new net GND: C901.2, C902.2, C903.2, R902.2, U901.10 (RESV), U901.11 (RESV), U901.2 (RESV), U901.3 (RESV), U901.6 (GND), U901.7 (RESV)
- new net I2C1_SCL: U901.13 (AP_SCL/AP_SCLK)
- new net I2C1_SDA: U901.14 (AP_SDA/AP_SDIO/AP_SDI)
- new net IMU_AD0: R902.1, R903.1, U901.1 (AP_SDO/AP_AD0)
- new net IMU_CS: R901.1, R904.1, U901.12 (AP_CS)
- new net IMU_CS_FB: R904.2
- new net IMU_INT1: U901.4 (INT1/INT)
- new net IMU_INT2: U901.9 (INT2/FSYNC/CLKIN)
- new net IMU_SDO_FB: R903.2
Other:
- note added: "IMU (Rev A) - design notes TDK ICM-42688-P (DS-000347 Rev 1.2) on I2C1 with the BQ25620 (pull-ups on the charger sheet), address 0x68. VDD = VDDIO = 3V3 (1.71-3.6 V); bypass per the datasheet BOM: 0.1 uF + 2.2 uF X7R on VDD, 10 nF X7R on VDDIO. RESV pins 2, 3, 7, 10, 11 to GND (allowed by Table 9). INT1 data-ready; pin 9 is INT2 (PIN9_FUNCTION reset default). SPI fallback: fit R903/R904 and move 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"

Commit message: hw: switch U401 to the E73 nRF52840 module
The MDBT53-P1M cannot be sourced in time for the Rev A order, while
the E73-2G4M08S1C is stocked at JLCPCB (ADR 0015).

The E73 holds its DC/DC inductors and decoupling, so L401/L402 and
C403/C404 are removed. The nRF52840 has no internal 32.768 kHz load,
so C405/C406 are fitted with 12 pF; the value is calculated and still
needs checking against the Product Specification. All 29 module GPIO
are used: CHG_STAT is no longer read by the MCU, and the UART pads,
spare GPIO pads and IMU SPI-fallback links are removed. Pins Ebyte
marks as low-frequency carry only analog inputs or slow signals.
Parts:
- removed R903, R904: DNP, Resistor_SMD:R_0402_1005Metric, symbol Device:R
Other:
- note added: "IMU (Rev A) - design notes TDK ICM-42688-P (DS-000347 Rev 1.2) on I2C1 with the BQ25620 (pull-ups on the charger sheet), address 0x68. VDD = VDDIO = 3V3 (1.71-3.6 V); bypass per the datasheet BOM: 0.1 uF + 2.2 uF X7R on VDD, 10 nF X7R on VDDIO. RESV pins 2, 3, 7, 10, 11 to GND (allowed by Table 9). INT1 data-ready; pin 9 is INT2 (PIN9_FUNCTION reset default). No SPI fallback: the E73 module chang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"
- note removed: "IMU (Rev A) - design notes TDK ICM-42688-P (DS-000347 Rev 1.2) on I2C1 with the BQ25620 (pull-ups on the charger sheet), address 0x68. VDD = VDDIO = 3V3 (1.71-3.6 V); bypass per the datasheet BOM: 0.1 uF + 2.2 uF X7R on VDD, 10 nF X7R on VDDIO. RESV pins 2, 3, 7, 10, 11 to GND (allowed by Table 9). INT1 data-ready; pin 9 is INT2 (PIN9_FUNCTION reset default). SPI fallback: fit R903/R904 and move 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"
