File: hardware/sheets/nfc.kicad_sch (KiCad schematic)
At the start: 13 parts, among them U1101 NT3H2111W0FHKH

Commit message: hw: remove unfitted parts and spare test points
Free routing room on the Rev A board:
- remove the eight DNP row pull-down arrays (RN709-RN716) and six DNP
  passive positions (C1103, R1005, R1104, R212, R213, R310)
- remove 19 test points outside the required set that had no room on
  the routed board

No net changes and no fitted-part changes, so the assembled board and
its BOM are the same. C1102 stays as the DNP NFC tuning position.
Parts:
- removed C1103: DNP, Capacitor_SMD:C_0402_1005Metric, symbol Device:C
- removed R1104: DNP, Resistor_SMD:R_0402_1005Metric, symbol Device:R
- removed TP1101: NFC_PWR, TestPoint:TestPoint_Pad_D1.0mm, symbol Connector:TestPoint
- removed TP1102: NFC_SDA, TestPoint:TestPoint_Pad_D1.0mm, symbol Connector:TestPoint
- removed TP1103: NFC_SCL, TestPoint:TestPoint_Pad_D1.0mm, symbol Connector:TestPoint
- removed TP1104: NFC_FD, TestPoint:TestPoint_Pad_D1.0mm, symbol Connector:TestPoint

Commit message: hw: align notes with the routed Rev A board
The sheet notes and docs still described parts that were removed from
the routed board. Update them:
- NFC: no dedicated test pads fit; probe VCC, SCL, SDA and FD at the
  0402 pads of C1101, R1101, R1102 and R1103
- VLED: no trim positions; a different setting means replacing R210
  (about 30-36.5 kOhm for 4.4-5.2 V with R211 at 4.7 kOhm, calculated)
- charger TS: no RT2 position; TI's network needs a resistor added
  across the NTC
- the test-point index lists the pads that remain

Also refresh the hardware README board section (outline, silkscreen,
DRC warnings) and link ADR 0016. No electrical changes.
Changed lines of the file:
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@@
 		(comment 2 "Schematic frozen for layout after review 2026-10-07; not for fabrication until the release gate")
 	)
-	(text "NFC (Rev A) - design notes\n\nNXP NT3H2111W0FHKH (Rev. 3.6; errata Rev. 4.1) on its own I2C bus (nRF52840 TWIM1, 100 kHz; TWIM0 serves I2C1). VCC, bus and FD pull-ups come from\nthe NFC_PWR GPIO (P1.00), on only during updates; RF reads are passive. VOUT (energy harvesting) unused.\nCoil: 30 x 25 mm, 6 turns, 0.4/0.3 mm, F.Cu with one In1.Cu crossover; no copper inside the coil region;\nbattery and magnets outside it (DEC-008). Resonance tuned down to about 14.5 MHz with C1102/C1103 (C0G).\nTest points on VCC, SDA, SCL, FD for bus and field-detect timing. Provisioning policy: docs/nfc.md. Nothing measured."
+	(text "NFC (Rev A) - design notes\n\nNXP NT3H2111W0FHKH (Rev. 3.6; errata Rev. 4.1) on its own I2C bus (nRF52840 TWIM1, 100 kHz; TWIM0 serves I2C1). VCC, bus and FD pull-ups come from\nthe NFC_PWR GPIO (P1.00), on only during updates; RF reads are passive. VOUT (energy harvesting) unused.\nCoil: 30 x 25 mm, 6 turns, 0.4/0.3 mm, F.Cu with one In1.Cu crossover; no copper inside the coil region;\nbattery and magnets outside it (DEC-008). Resonance tuned down to about 14.5 MHz with C1102 (C0G, DNP).\nNo NFC test pads (no room): probe C1101 (VCC), R1101 (SCL), R1102 (SDA), R1103 (FD). Provisioning policy: docs/nfc.md. Nothing measured."
 		(exclude_from_sim no)
 		(at 50.8 152.4 0)
