File: hardware/sheets/microphone.kicad_sch (KiCad schematic)
At the start: 0 parts

Commit message: hw: draw UI, IMU, microphone and NFC sheets
IMU: ICM-42688-P on the shared I2C1 bus at 0x68, bypassed as TDK's
application circuit specifies, reserved pins to ground, and unfitted
links for the SPI fallback.

Microphone: SPH0641LM4H-1 with a C0G bypass capacitor (Knowles advises
against class 2 dielectrics next to the part), a 0 ohm supply link for
current measurement, series options on clock and data, and SELECT to
ground.

NFC: NT3H2111W0FHKH powered from the NFC_PWR GPIO with its bus and
field-detect pull-ups, the PCB coil as a non-BOM part, two unfitted
tuning capacitor positions and test points for bus timing.

UI: two tact switches to ground with unfitted external pull-ups and a
red status LED.

The labels these sheets connect no longer need ERC exclusions. NFC_PWR
gets a reviewed exclusion: a GPIO drives the tag supply by design.
Parts:
- added C1001: 100nF C0G, Capacitor_SMD:C_1206_3216Metric, symbol Device:C
- added MK1001: SPH0641LM4H-1, smart-led-badge:Knowles_LGA-5_3.5x2.65mm_Hole0.8mm, symbol Sensor_Audio:SPH0641LU4H-1
- added R1001, R1002, R1003, R1004: 0, Resistor_SMD:R_0402_1005Metric, symbol Device:R
- added R1005: DNP, Resistor_SMD:R_0402_1005Metric, symbol Device:R
- added TP1001: PDM_CLK, TestPoint:TestPoint_Pad_D1.0mm, symbol Connector:TestPoint
- added TP1002: PDM_DIN, TestPoint:TestPoint_Pad_D1.0mm, symbol Connector:TestPoint
Connections:
- new net +3V3: R1001.1
- new net GND: C1001.2, MK1001.3 (GND), R1004.2
- new net MIC_SEL: MK1001.2 (SEL), R1004.1, R1005.1
- new net MIC_VDD: C1001.1, MK1001.5 (VDD), R1001.2, R1005.2
- new net PDM_CLK: R1002.1, TP1001.1
- new net PDM_CLK_MIC: MK1001.4 (CLOCK), R1002.2
- new net PDM_DIN: R1003.2, TP1002.1
- new net PDM_DIN_MIC: MK1001.1 (DATA), R1003.1
Other:
- note added: "Microphone (Rev A) - design notes Knowles SPH0641LM4H-1 (Rev D) PDM, bottom port: 1.6-3.6 V; modes by clock (sleep < 280 kHz, low power 351-815 kHz, normal 1.0-4.8 MHz). SELECT = GND: firmware samples the mono channel on the PDM_CLK rising edge (nRF PDM EDGE). Bypass C0G at the Vdd pin (Knowles: no class 2 dielectrics near the mic). R1001 links 3V3 for current measurement. PCB acoustic hole 0.8 m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"

Commit message: hw: apply layout footprint and test-point changes to the schematic
The matrix LEDs use the KENTO-pattern footprint, L1101 the PCB coil,
MK1001 the 0.6 mm hole footprint and J301 the project HRO copy.

Removes test points that duplicate others: TP303 and TP304, TP208 and
TP506, and TP501-TP503, whose signals are on the SWD header. Also
removes H1304, which the carrier does not use. Rail and GND test points
move to 0.8 mm pads.

nRESET now connects only the header's open-collector pin and the module
input. ERC reports that as not driven, so the error is excluded: the
nRF5340 has an internal pull-up on reset.
Parts:
- MK1001: footprint smart-led-badge:Knowles_LGA-5_3.5x2.65mm_Hole0.8mm -> smart-led-badge:Knowles_LGA-5_3.5x2.65mm_Hole0.6mm
Changed lines of the file:
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@@
 			)
 		)
-		(property "Footprint" "smart-led-badge:Knowles_LGA-5_3.5x2.65mm_Hole0.8mm"
+		(property "Footprint" "smart-led-badge:Knowles_LGA-5_3.5x2.65mm_Hole0.6mm"
 			(at 101.6 88.9 0)
 			(hide yes)

Commit message: hw: lay out and route the Rev A board (#29)
* hw: add fab-layer references to custom footprints

Show each part's reference on F.Fab so the assembly drawing used for
bring-up and rework labels the custom parts the same way as the KiCad
library parts. Copper, courtyards and silkscreen are unchanged.

* hw: join the NFC coil's twin pad-2 ends as a jumper

The coil's inner and outer pad-2 ends are connected by footprint copper
(the In1 crossover), which KiCad does not count as a connection, so
NFC_LB stayed unrouted. Treat the duplicate pad numbers as a jumper.
The pad 1/2 net tie is unchanged.

* hw: remove unfitted parts and spare test points

Free routing room on the Rev A board:
- remove the eight DNP row pull-down arrays (RN709-RN716) and six DNP
  passive positions (C1103, R1005, R1104, R212, R213, R310)
- remove 19 test points outside the required set that had no room on
  the routed board

No net changes and no fitted-part changes, so the assembled board and
its BOM are the same. C1102 stays as the DNP NFC tuning position.

* hw: lay out and route the Rev A board

Place and route the 118 x 76 mm four-layer board: the 32 x 32 matrix at
45 degrees on the west, the row drivers in a column beside it, and the
power, charger, NFC, IMU, microphone and E73 module on the east. In1 is
a GND plane kept solid under the regulators, charger and module; a few
low-current signals cross it elsewhere where no other layer had room.
The board uses the JLC04161H-7628 stack-up, tented vias and
0.45/0.2 mm minimum vias.

Add release silkscreen: battery polarity at J302 on both faces,
test-point net names (front where they fit, rear behind each pad),
orientation-independent control marks, the board name and a designer
monogram on the NFC coil.

DRC and schematic parity are clean. Nothing is measured yet: charger,
USB, matrix timing, RF and NFC tuning remain bring-up checks. The README
and hardware docs now give the 118 x 76 mm outline.

* hw: move three vias out of component pads

The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
Parts:
- removed R1005: DNP, Resistor_SMD:R_0402_1005Metric, symbol Device:R
Changed lines of the file:
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@@
-	(wire
-		(pts
-			(xy 162.56 120.65) (xy 162.56 118.11)
-		)
-		(stroke
-			(width 0)
-			(type default)
-		)
-	)
 	(wire
 		(pts
@@
 	(wire
 		(pts
-			(xy 162.56 128.27) (xy 162.56 130.81)
-		)
-		(stroke
-			(width 0)
-			(type default)
-		)
-	)
-	(wire
-		(pts
 			(xy 76.2 59.69) (xy 76.2 62.23)
 		)
@@
 			(width 0)
 			(type default)
-		)
-	)
-	(label "MIC_VDD"
-		(at 162.56 130.81 270)
-		(effects
-			(font
-				(size 1.27 1.27)
-			)
-			(justify right bottom)
 		)
 	)
@@
 			)
 			(justify right bottom)
-		)
-	)
-	(label "MIC_SEL"
-		(at 162.56 118.11 90)
-		(effects
-			(font
-				(size 1.27 1.27)
-			)
-			(justify left bottom)
 		)
 	)
@@
 					(unit 1)
 				)
-			)
-		)
-	)
-	(symbol
-		(lib_id "Device:R")
-		(at 162.56 124.46 0)
-		(unit 1)
-		(body_style 1)
-		(exclude_from_sim no)
-		(in_bom yes)
-		(on_board yes)
-		(in_pos_files yes)
-		(dnp yes)
-		(property "Reference" "R1005"
-			(at 165.1 123.19 0)
-			(show_name no)
-			(do_not_autoplace no)
-			(effects
-				(font
-					(size 1.27 1.27)
-				)
-				(justify left)
-			)
-		)
-		(property "Value" "DNP"
-			(at 165.1 125.73 0)
-			(show_name no)
-			(do_not_autoplace no)
-			(effects
-				(font
-					(size 1.27 1.27)
-				)
-				(justify left)
-			)
-		)
-		(property "Footprint" "Resistor_SMD:R_0402_1005Metric"
-			(at 162.56 124.46 0)
-			(hide yes)
-			(show_name no)
-			(do_not_autoplace no)
-			(effects
-				(font
-					(size 1.27 1.27)
-				)
-			)
-		)
-		(property "Datasheet" ""
-			(at 162.56 124.46 0)
-			(hide yes)
-			(show_name no)
-			(do_not_autoplace no)
-			(effects
-				(font
-					(size 1.27 1.27)
-				)
-			)
-		)
-		(property "Description" "Resistor"
-			(at 162.56 124.46 0)
-			(hide yes)
-			(show_name no)
-			(do_not_autoplace no)
-			(effects
-				(font
-					(size 1.27 1.27)
-				)
-			)
-		)
-		(property "Note" "SELECT high option (fit instead of R1004)"
-			(at 162.56 124.46 0)
-			(hide yes)
-			(show_name no)
-			(do_not_autoplace no)
-			(effects
-				(font
-					(size 1.27 1.27)
-				)
-			)
-		)
-		(pin "1"
-		)
-		(pin "2"
-		)
-		(instances
-			(project "smart-led-badge"
-				(path "/fefc8d4a-8637-4143-b210-9149e35f9884/aa96d21e-cc37-4bd6-a260-2721aeab775d"
-					(reference "R1005")
-					(unit 1)
-				)
